File: flight-subsystem-designs/gnc/GPS-RadioPCB/SpaceManiacPCB Kopie.kicad_sch (KiCad schematic)
At the start: 39 parts, among them Q1 EPC2014C, U1 LMK1C1104PWR

Commit message: For Zumi Schematik Review
Parts:
- removed D1, D2, D3, D4, D5: TVS5B5CL, Diode_SMD:Nexperia_DSN1608-2_1.6x0.8mm, symbol Diode:PTVS5V0Z1USK
- removed R1: 10k, Resistor_SMD:R_0402_1005Metric, symbol Device:R_Small
- removed R3, R4: 120 Ohm, Resistor_SMD:R_0402_1005Metric, symbol Device:R
- added R2: 300k, Resistor_SMD:R_0402_1005Metric, symbol Device:R_Small
- C5, C6, C7: footprint Capacitor_SMD:C_0402_1005Metric -> Capacitor_SMD:C_0603_1608Metric
Connections:
- net CAN_H is gone; now on net CAN+: H1.3 (Pin_3), H3.26 (Pin_26), H4.26 (Pin_26)
- net CAN_L is gone; now on net CAN-: H1.1 (Pin_1), H3.28 (Pin_28), H4.28 (Pin_28)
- net CLK_0: now also H1.52 (Pin_52); no longer H2.16 (Pin_16)
- net CLK_1: now also H1.50 (Pin_50); no longer H2.15 (Pin_15)
- net CLK_2: now also H1.51 (Pin_51); no longer H2.17 (Pin_17)
- net GND: now also C4.2, R2.1; no longer C4.1
- net PWR_Fanout: now also C4.1, U1.2 (1G), R2.2; no longer C4.2
- net CAN+: now reaches H4.25 (Pin_25)
- net CAN-: now reaches H4.27 (Pin_27)
- removed net RAW_BATT: H1.6 (Pin_6), H1.8 (Pin_8), H3.1 (Pin_1), H3.2 (Pin_2), H4.1 (Pin_1), H4.2 (Pin_2)
- no-connect marks 160 -> 161
Other:
- moved on the sheet: C4, C5, C6, C7, D6, D7, H10, H11, H12, H13, H14, H15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
