File: flight-subsystem-designs/payload/RealQuadcellAmp/RealQuadcellAmp.kicad_sch (KiCad schematic)
At the start: 52 parts, among them J1 Screw_Terminal_01x02, J2 Conn_01x04_Pin, J3 Conn_01x04_Pin, U1 LM2904, U2 LM2904, U3 LM2904, U4 LM2904, U6 LM2904

Commit message: fix: added ucsp schematic template
Other:
- company: (none) -> UChicago Space Program
- title: (none) -> Quadcell Amplifier
- moved on the sheet: C1, C10, C12, C3, C4, C6, C7, C9, R1, R10, R12, R13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
