File: flight-subsystem-designs/payload/RealQuadcellAmp/RealQuadcellAmp.kicad_sch (KiCad schematic)
At the start: 52 parts, among them J1 Screw_Terminal_01x02, J2 Conn_01x04_Pin, J3 Conn_01x04_Pin, U1 LM2904, U2 LM2904, U3 LM2904, U4 LM2904, U6 LM2904

Commit message: feat: small tweaks for schematic review
Parts:
- R10, R14, R2, R6: value 100 MΩ -> 1 MΩ
Changed lines of the file:
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@@
 			)
 		)
-		(property "Value" "100 MΩ"
+		(property "Value" "1 MΩ"
 			(at 69.85 78.7399 0)
 			(effects
@@
 			)
 		)
-		(property "Value" "100 MΩ"
+		(property "Value" "1 MΩ"
 			(at 72.39 46.9899 0)
 			(effects
@@
 			)
 		)
-		(property "Value" "100 MΩ"
+		(property "Value" "1 MΩ"
 			(at 70.612 96.52 0)
 			(effects
@@
 			)
 		)
-		(property "Value" "100 MΩ"
+		(property "Value" "1 MΩ"
 			(at 72.39 29.2099 0)
 			(effects
