File: flight-subsystem-designs/cdh/flight-computer/OBCV6.1(WIP).kicad_sch (KiCad schematic)
At the start: 34 parts, among them J1 Conn_01x03, J2 Conn_01x03, J3 Conn_01x03, J4 Conn_01x03, J5 Conn_01x03, J6 Conn_01x03, U1 BEAGLEBONEBLACK, U2 Payload, U3 TCAN337G, U4 MCP7940N-xSN, U5 W25N01GVZEIG_TR, U6 MAX706RESA+T, U7 TMP36xS

Commit message: fix: added ucsp header to obc and deleted duplicate schematic
Parts:
- removed R8, R9: 10, Resistor_SMD:R_0805_2012Metric_Pad1.20x1.40mm_HandSolder, symbol Device:R
- removed U5: W25N01GVZEIG_TR, W25N01GVZEIG_TR:SON127P800X600X80-9N, symbol W25N01GVZEIG_TR:W25N01GVZEIG_TR
Connections:
- net NANDWPI: no longer names the net of U1.P8_29 (GPIO2_23)
- net NAND_HOLD: no longer names the net of U1.P8_30 (GPIO2_25)
Other:
- company: (none) -> University of Chicago Space Program
- title: (none) -> On-board Computer
- moved on the sheet: U1
