File: flight-subsystem-designs/cdh/flight-computer/Ian OBC Recreation/Ian OBC Recreation.kicad_sch (KiCad schematic)
At the start: 42 parts, among them J8 Conn_02x26_Odd_Even, Q1 AON6411, Q2 AON6411, U1 BEAGLEBONEBLACK, U2 TPS2400DBVR, U3 TCAN337G, U4 MCP7940N-xSN, U5 ADM3485EARZ, U6 MAX706RESA+T, U7 TMP36xS, U8 TPS2400DBVR

Commit message: feat: small tweaks for schematic review
Other:
- note added: "RS485 BACKUP CAN"
- note removed: "RS45 BACKUP CAN"
Changed lines of the file:
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@@
 		)
 	)
-	(text "RS45 BACKUP CAN"
+	(text "RS485 BACKUP CAN"
 		(exclude_from_sim no)
 		(at 380.492 177.038 0)
