File: flight-subsystem-designs/cdh/flight-computer/Ian OBC Recreation/Ian OBC Recreation.kicad_sch (KiCad schematic)
At the start: 47 parts, among them Q1 AON6411, Q2 AON6411, U1 BEAGLEBONEBLACK, U2 TPS2400DBVR, U3 TCAN337G, U4 MCP7940N-xSN, U5 ADM3485EARZ, U6 MAX706RESA+T, U7 TMP36xS, U8 TPS2400DBVR

Commit message: feat improvement
Parts:
- removed Q1, Q2: AON6411, Package_DFN_QFN:AO_DFN-8-1EP_5.55x5.2mm_P1.27mm_EP4.12x4.6mm, symbol Transistor_FET:AON6411
- removed TP3, TP4, TP5, TP6: TestPoint, TestPoint:TestPoint_THTPad_D3.0mm_Drill1.5mm, symbol Connector:TestPoint
- removed U2, U8: TPS2400DBVR, Footprints:SOT95P280X145-5N, symbol TPS2400DBVR:TPS2400DBVR
- added D1: BAT54CW, Package_TO_SOT_SMD:SOT-323_SC-70, symbol Diode:BAT54CW
- C12, C7, C8, C9: footprint (none) -> Capacitor_SMD:C_0805_2012Metric_Pad1.18x1.45mm_HandSolder
Connections:
- net 3V3IN: no longer C12.1, C8.1, H6.27 (Pin_27)
- net 5VIN: no longer C7.1, C9.1, H6.25 (Pin_25)
- net DCAN1RX: now also U1.P9_20 (I2C2_SDA); no longer U1.P9_24 (UART1_TXD)
- net DCAN1TX: now also U1.P9_19 (I2C2_SCL); no longer U1.P9_26 (UART1_RXD)
- net SYSRST: no longer H5.14 (Pin_14)
- net SYS_5V: now also C7.1, C9.1, H6.25 (Pin_25)
- net VDD_3V3B: now also C12.1, C8.1, H6.27 (Pin_27), D1.2; no longer XTAL1.4 (Vdd)
- net PPS: now reaches U1.P8_3 (GPIO1_6)
- net PPS: now also H5.14 (Pin_14)
- net at BT1.1 (+), U4.3 (VBAT): now also D1.1
- new net OSCVDD: D1.3, XTAL1.4 (Vdd)
- no-connect marks 96 -> 93
Other:
- note added: "This Space Shall be Left Empty in Honor of My Late Overvoltage Circuit that Zumi Killed"
- note removed: "OVERVOLTAGE PROTECTION"

Commit message: Updated to match current ICD on Drive
Parts:
- added D2: 5V, LED_SMD:LED_0805_2012Metric, symbol Device:LED
- added D3: 3V3, LED_SMD:LED_0805_2012Metric, symbol Device:LED
Connections:
- net 3V3IN is gone; now on net VDD_3V3B: H6.28 (Pin_28)
- net 5VIN is gone; now on net SYS_5V: H6.26 (Pin_26)
- net 5V_S_EN is gone; now on net SPI_DO: H5.31 (Pin_31)
- net BURN1_N is gone; now on net SPI_CSO: H5.28 (Pin_28)
- net BURN2_N is gone; now on net SPI_D1: H5.30 (Pin_30)
- net BURN_IN is gone; now on net SPI_SCLK: H5.29 (Pin_29)
- net GPIO1_27 is gone; now on net DGND: H5.36 (Pin_36)
- net SEL_MODE is gone; now on net PPS: U1.P8_40 (GPIO2_13)
- net CAN_FAULT: now also U1.P8_37 (UART5_TXD); no longer U1.P8_25 (GPIO1_0)
- net DGND: now also H5.34 (Pin_34), H5.6 (Pin_6), H6.4 (Pin_4), H6.6 (Pin_6), D2.1 (K), D3.1 (K); no longer H5.10 (Pin_10), H5.12 (Pin_12), H6.31 (Pin_31), H6.32 (Pin_32)
- net GPIO1_15: no longer H5.17 (Pin_17)
- net GPIO2_1: no longer H5.48 (Pin_48)
- net GPIO2_11: no longer H5.18 (Pin_18)
- net GPIO2_22: no longer H5.50 (Pin_50)
- net GPIO2_8: no longer H5.16 (Pin_16)
- net GPIO2_9: no longer H5.34 (Pin_34)
- net MRV: now also U1.P9_11 (UART4_RXD); no longer U1.P8_23 (GPIO1_4)
- net PPS: no longer U1.P8_3 (GPIO1_6)
- net RTCC_MFP: now also U1.P9_13 (UART4_TXD); no longer U1.P8_22 (GPIO1_5)
- net SYS_5V: now also D2.2 (A)
- net UART_RX: no longer H5.35 (Pin_35)
- net UART_TX: no longer H5.33 (Pin_33)
- net VDD_3V3B: now also D3.2 (A)
- net GPIO1_17: now reaches U1.P9_23 (GPIO1_17)
- net GPIO1_17: now also U5.2 (RE*), U5.3 (DE)
- net UART2_TX: now reaches U1.P9_24 (UART1_TXD)
- net UART2_TX: now also H5.33 (Pin_33)
- net UART2_RX: now reaches U1.P9_26 (UART1_RXD)
- net UART2_RX: now also H5.35 (Pin_35)
- net SPI_CSO: now reaches U1.P9_28 (SPI1_CS0)
- net SPI_DO: now reaches U1.P9_29 (SPI1_D0)
- net SPI_D1: now reaches U1.P9_30 (SPI1_D1)
- net SPI_SCLK: now reaches U1.P9_31 (SPI1_SCLK)
- net VBAT: now reaches H6.45 (Pin_45)
- net VBAT: now also H6.46 (Pin_46)
- net 3V3_S_EN: no longer names the net of H5.27 (Pin_27)
- net BATT_FAULT: no longer names the net of H5.22 (Pin_22)
- net BATT_HEAT_EN: no longer names the net of H5.13 (Pin_13)
- net BAT_BRD_TMP: no longer names the net of H6.1 (Pin_1)
- net CHRG: no longer names the net of H5.24 (Pin_24)
- removed net GPIO1_1: U1.P8_24 (GPIO1_1), U5.2 (RE*), U5.3 (DE)
- net GPIO1_26: no longer names the net of H5.15 (Pin_15)
- net NANDWPI: no longer names the net of U1.P8_29 (GPIO2_23)
- net NAND_HOLD: no longer names the net of U1.P8_30 (GPIO2_25)
- net PDU_TMP: no longer names the net of H6.2 (Pin_2)
- net SBWTCK: no longer names the net of H5.52 (Pin_52)
- net SBWTDI0: no longer names the net of H5.51 (Pin_51)
- net SOL_SHDN: no longer names the net of H5.26 (Pin_26)
- net SWITCH_MODE_SEL: no longer names the net of H5.25 (Pin_25)
- net SWITCH_SHUTDOWN: no longer names the net of H5.46 (Pin_46)
- no-connect marks 93 -> 108
Other:
- note added: "LED INDICATORS"
