File: Avionics/PowerDistribution/PowerDistribution.kicad_pcb (KiCad board)
At the start: 4 copper layers, 90.2 x 96 mm, 135 parts, among them J1 Conn_02x26_Odd_Even, J11 Conn_01x04, J12 Conn_01x04, J13 Conn_01x04, J15 Conn_01x02, J2 Conn_02x26_Odd_Even, J3 Conn_01x02, J4 Conn_01x02, J5 Conn_01x02, J6 Conn_01x02, J8 Conn_01x02, Q1 BC848ALT1G, Q2 IRLML2803PBFCT, Q3 IRLML2803PBFCT, U1 LT8610, U12 LTM8062AIV-PBF, U16 INA219AxD, U17 INA219AxD, U18 INA219AxD, U2 LT8610, U21 INA219AxD, U6 LT8610

Commit message: feat: 3.1
Parts:
- removed R1: 100k, Resistor_SMD:R_0603_1608Metric
- removed R31: 549k, Resistor_SMD:R_0603_1608Metric
- C12, C3: footprint Capacitor_SMD:C_0805_2012Metric -> Capacitor_SMD:C_1206_3216Metric
- C24: value 47uF -> 68uF; footprint Capacitor_SMD:C_0805_2012Metric -> Capacitor_SMD:C_1206_3216Metric
- R33: value 2m -> 10m
- R34: value 549k -> 642k
- R40: value 459k -> 412k
- R43, R52, R55: value 2m -> 40m
- moved C24 0.66 mm to (209.6, 129.8)
- moved C3 0.62 mm to (191.4, 129.9)
- moved C12 0.58 mm to (209.5, 110.9)
- turned C35 to 0 degrees
Connections:
- C35 pad 1: GND -> VBATT
- C35 pad 2: VBATT -> GND
- J1 pad 36: /ADJ -> unconnected-(J1-Pin_36-Pad36)
- J1 pad 38: /BATT_THERM_R -> unconnected-(J1-Pin_38-Pad38)
Routing:
- net /BATT_THERM_R: track 33.5 -> 0.00 mm
- net /ADJ: track 35.0 -> 3.36 mm, vias 2 -> 0
- net EDFA_5V: track 36.9 -> 35.2 mm, vias 8 -> 7
Other:
- board text added: "rev. 3.1, 04.14.26"
- board text removed: "rev. 3.0.0, 06.30.25"
