File: Avionics/PowerDistribution/PowerDistribution.kicad_sch (KiCad schematic)
At the start: 134 parts, among them J1 Conn_02x26_Odd_Even, J11 Conn_01x04, J12 Conn_01x04, J13 Conn_01x04, J15 Conn_01x02, J2 Conn_02x26_Odd_Even, J3 Conn_01x02, J4 Conn_01x02, J5 Conn_01x02, J6 Conn_01x02, J8 Conn_01x02, Q1 BC848ALT1G, Q2 IRLML2803PBFCT, Q3 IRLML2803PBFCT, U1 LT8610, U12 LTM8062AIV-PBF, U16 INA219AxD, U17 INA219AxD, U18 INA219AxD, U2 LT8610, U21 INA219AxD, U6 LT8610

Commit message: feat: 3.1
Parts:
- removed R1: 100k, Resistor_SMD:R_0603_1608Metric, symbol Device:R
- removed R31: 549k, Resistor_SMD:R_0603_1608Metric, symbol Device:R
- C12, C3: footprint Capacitor_SMD:C_0805_2012Metric -> Capacitor_SMD:C_1206_3216Metric
- C24: value 47uF -> 68uF; footprint Capacitor_SMD:C_0805_2012Metric -> Capacitor_SMD:C_1206_3216Metric
- L3: value 4.7uH -> 10uH
- R33: value 2m -> 10m
- R34: value 549k -> 642k
- R40: value 459k -> 412k
- R43, R52, R55: value 2m -> 40m
Connections:
- net ADJ: no longer J1.36 (Pin_36)
- net GND: now also C35.2; no longer C35.1
- net VBATT: now also C35.1; no longer C35.2
- net BATT_THERM_R: no longer names the net of J1.38 (Pin_38)
- no-connect marks 68 -> 70
Other:
- moved on the sheet: C35, R34, R40
