File: flight-subsystem-designs/power/batteryboard-v01b/batteryboard.kicad_pcb (KiCad board)
At the start: 2 copper layers, 90.2 x 95.9 mm, 26 parts, among them J1 KEYSTONE-1042, J2 KEYSTONE-1042, J3 KEYSTONE-1042, J4 KEYSTONE-1042, J5 15453216, Q1 IRF7458, Q2 IRF7458, U1 R5460N233AF

Commit message: battboard: v4.0.0 PyCubed Edition
Parts:
- added G***: LOGO, LOGO, B.Cu at (138.9, 108.6)
- added J6: Left Header, Connector_PinSocket_2.54mm:PinSocket_1x04_P2.54mm_Vertical, F.Cu at (58.5, 71.8)
- added J7: Right Header, Connector_PinSocket_2.54mm:PinSocket_1x04_P2.54mm_Vertical, F.Cu at (143.8, 126.0)
- moved R1 0.81 mm to (115.8, 72.7), turned to -90 degrees
- moved R3 0.17 mm to (122.1, 78.0)
Connections:
- J5 pad 10: unconnected-(J5-Pad10) -> Net-(J6-Pin_3)
- J5 pad 11: unconnected-(J5-Pad11) -> Net-(J6-Pin_2)
- J5 pad 12: unconnected-(J5-Pad12) -> Net-(J6-Pin_1)
- J5 pad 13: unconnected-(J5-Pad13) -> Net-(J7-Pin_4)
- J5 pad 14: unconnected-(J5-Pad14) -> Net-(J7-Pin_3)
- J5 pad 15: unconnected-(J5-Pad15) -> Net-(J7-Pin_2)
- J5 pad 16: unconnected-(J5-Pad16) -> Net-(J7-Pin_1)
- J5 pad 9: unconnected-(J5-Pad9) -> Net-(J6-Pin_4)
Routing:
- net Net-(J7-Pin_3): track 0.00 -> 87.2 mm
- net Net-(J7-Pin_4): track 0.00 -> 86.5 mm
- net Net-(J7-Pin_2): track 0.00 -> 73.1 mm
- net Net-(J7-Pin_1): track 0.00 -> 71.2 mm
- net Net-(J6-Pin_3): track 0.00 -> 42.2 mm
- net Net-(J6-Pin_1): track 0.00 -> 42.0 mm
- net Net-(J6-Pin_4): track 0.00 -> 36.7 mm
- net Net-(J6-Pin_2): track 0.00 -> 36.3 mm
- net PACK-: track 63.2 -> 65.1 mm
- net PACK+: track 29.6 -> 28.1 mm, vias 16 -> 18
- net /DOUT: track 67.1 -> 67.8 mm
- net BM: track 89.0 -> 89.7 mm
- net B-: track 16.8 -> 16.9 mm, vias 14 -> 22
Other:
- board text added: "AVIONICS"
- board text added: "Conn. Pins (L to R): 12, 11, 10, 9"
- board text added: "Conn. Pins (L to R): 16, 15, 14, 13"
- board text added: "PULSE-A"
- board text added: "battery pack"
- board text added: "rev. 4.0.0, 2026-04-06"
- board text added: "{dblquote}Back to Basics{dblquote}"
- board text added: "{dblquote}We're so back{dblquote} -Dylan H"
