File: flight-subsystem-designs/power/batteryboard-v01b/batteryboard.kicad_sch (KiCad schematic)
At the start: 26 parts, among them J1 KEYSTONE-1042, J2 KEYSTONE-1042, J3 KEYSTONE-1042, J4 KEYSTONE-1042, J5 15453216, Q1 IRF7458, Q2 IRF7458, U1 R5460N233AF

Commit message: battboard: v4.0.0 PyCubed Edition
Parts:
- added J6: Left Header, Connector_PinSocket_2.54mm:PinSocket_1x04_P2.54mm_Vertical, symbol Connector_Generic:Conn_01x04
- added J7: Right Header, Connector_PinSocket_2.54mm:PinSocket_1x04_P2.54mm_Vertical, symbol Connector_Generic:Conn_01x04
Connections:
- net at J5.10: now also J6.3 (Pin_3)
- net at J5.11: now also J6.2 (Pin_2)
- net at J5.12: now also J6.1 (Pin_1)
- net at J5.13: now also J7.4 (Pin_4)
- net at J5.14: now also J7.3 (Pin_3)
- net at J5.15: now also J7.2 (Pin_2)
- net at J5.16: now also J7.1 (Pin_1)
- net at J5.9: now also J6.4 (Pin_4)
- no-connect marks 12 -> 4
