File: flight-subsystem-designs/cdh/flight-computer/OBCV7/_autosave-OBCV7.kicad_sch (KiCad schematic)
At the start: 43 parts, among them U1 BEAGLEBONEBLACK, U3 TCAN337G, U4 MCP7940N-xSN, U5 ADM3485EARZ, U6 MAX706RESA+T, U7 TMP36xS

Commit message: New Board Version with better Signal Integrity
Connections:
- net CAN_FAULT: now also U1.P8_14 (GPIO0_26); no longer U1.P8_37 (UART5_TXD)
Other:
- moved on the sheet: BT1, C1, C10, C11, C12, C2, C3, C4, C5, C6, C7, C8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
