File: flight-subsystem-designs/cdh/flight-computer/OBCV7/_autosave-OBCV7.kicad_sch (KiCad schematic)
At the start: 44 parts, among them U1 BEAGLEBONEBLACK, U3 TCAN337G, U4 MCP7940N-xSN, U5 ADM3485EARZ, U6 MAX706RESA+T, U7 TMP36xS

Commit message: Perhaps technology is hubris manifest
Parts:
- C5: value 5nF -> 10nF
Changed lines of the file:
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@@
 			)
 		)
-		(property "Value" "5nF"
+		(property "Value" "10nF"
 			(at 370.84 66.04 90)
 			(effects
