File: flight-subsystem-designs/cdh/flight-computer/OBCV7/OBCV7.kicad_pcb (KiCad board)
At the start: 4 copper layers, 90.3 x 95.9 mm, 45 parts, among them U1 BEAGLEBONEBLACK, U3 TCAN337G, U4 MCP7940N-xSN, U5 ADM3485EARZ, U6 MAX706RESA+T, U7 TMP36xS

Commit message: Hopefully Final-ish Board
Parts:
- added 3V3: TestPoint, TestPoint:TestPoint_THTPad_D3.0mm_Drill1.5mm, F.Cu at (121.7, 122.6)
- renumbered TP3 to GND, TP2 to OSC, TP1 to WDO
Connections:
- C7 pad 1: SYS_5V -> VDD_5V
- C9 pad 1: SYS_5V -> VDD_5V
- D2 pad 2: SYS_5V -> VDD_5V
- U1 pad P9_5: SYS_5V -> VDD_5V
- U1 pad P9_6: SYS_5V -> VDD_5V
- U1 pad P9_7: SYS_5V -> SYS_5V_1
Routing:
- net SYS_5V: track 164.2 -> 119.4 mm, vias 2 -> 0
- net VDD_5V: track 0.00 -> 29.3 mm, vias 0 -> 2
- net Net-(C11-Pad1): track 184.3 -> 200.9 mm
- net /UART_RX: track 102.2 -> 100.6 mm
- net /UART2_RX: track 95.6 -> 94.0 mm
- net /Temp: track 62.7 -> 61.2 mm
- net /SPI_DO: track 78.0 -> 76.5 mm
- net /I2C_SCL: track 171.1 -> 170.0 mm
- net /SPI_SCLK: track 113.0 -> 114.0 mm
- net /I2C_SDA: track 260.0 -> 259.0 mm
- net /SPI_D1: track 94.5 -> 93.7 mm
- net /UART2_TX: track 88.8 -> 88.0 mm
Other:
- outline, holes or cut-outs redrawn

Commit message: Final Board (Hopefully)
Routing:
- net Net-(BT1-+): track 92.9 -> 98.8 mm
- net /GPIO1_17: track 39.0 -> 41.9 mm
- net Net-(C4-Pad1): track 16.8 -> 19.4 mm, vias 3 -> 2
- net /RTCC_MFP: track 33.8 -> 35.7 mm
- net /I2C_SCL: track 170.0 -> 171.8 mm
- net /UART_TX: track 90.2 -> 90.8 mm
Other:
- outline, holes or cut-outs redrawn
