File: flight-subsystem-designs/cdh/flight-computer/OBCV7/OBCV7.kicad_pcb (KiCad board)
At the start: 4 copper layers, 90.3 x 95.9 mm, 48 parts, among them U1 BEAGLEBONEBLACK, U3 TCAN337G, U4 MCP7940N-xSN, U5 ADM3485EARZ, U6 MAX706RESA+T, U7 TMP36xS

Commit message: watchdog corrections and other shi
Parts:
- added C13: 100nf, Capacitor_SMD:C_0805_2012Metric_Pad1.18x1.45mm_HandSolder, F.Cu at (154.9, 101.6)
- added C14: 100nf, Capacitor_SMD:C_0805_2012Metric_Pad1.18x1.45mm_HandSolder, F.Cu at (136.9, 104.3)
- added S1: EG1215AA, Footprints:SW_EG1215AA, F.Cu at (105.5, 120.0)
- U6: value MAX706RESA+T -> MAX706ARESA+T
- moved 3V3 17.7 mm to (116.2, 120.6)
- moved WDO1 16.8 mm to (120.7, 120.6)
- moved GND1 4.43 mm to (111.8, 120.6)
- moved OSC1 4.43 mm to (111.8, 115.5)
Connections:
- U1 pad P9_11: /MRV -> unconnected-(U1-UART4_RXD-PadP9_11)
- U1 pad P9_4: VDD_3V3B_1 -> VDD_3V3B
- U6 pad 2: /3V3 -> VDD_3V3B
- U6 pad 6: /GPIO3_20 -> Net-(U6-WDI)
Routing:
- net Net-(U6-WDI): track 0.00 -> 58.4 mm
- net /GPIO3_20: track 62.7 -> 22.8 mm
- net VDD_3V3B: track 0.00 -> 26.2 mm
- net /MRV: track 83.4 -> 63.5 mm
- net GND: track 157.7 -> 163.2 mm
- net /3V3: track 94.4 -> 89.8 mm, vias 9 -> 8
- net Net-(U4-X1): track 51.5 -> 47.1 mm
Other:
- board text added: "FOR TESTING PURPOSES: POWER 5V BEFORE 3V3 CATASTROPHIC BACKPOWERING IF NOT FOLLOWED"
- board text added: "Rev. 7.0.0 - 9.2.26 - Gianni Alberico"
- board text removed: "Rev. 7.0.0 - 8.6.26 - Gianni Alberico"
