File: flight-subsystem-designs/cdh/flight-computer/OBCV7/OBCV7.kicad_sch (KiCad schematic)
At the start: 44 parts, among them U1 BEAGLEBONEBLACK, U3 TCAN337G, U4 MCP7940N-xSN, U5 ADM3485EARZ, U6 MAX706RESA+T, U7 TMP36xS

Commit message: perhaps technology is hubris manifest
Parts:
- removed R10, R4, R5: 62, Resistor_SMD:R_0805_2012Metric_Pad1.20x1.40mm_HandSolder, symbol Device:R
- removed R11: 10k, Resistor_SMD:R_0805_2012Metric_Pad1.20x1.40mm_HandSolder, symbol Device:R
- added R12: 150, LED_SMD:LED_0805_2012Metric, symbol Device:R
- added R13: 62, LED_SMD:LED_0805_2012Metric, symbol Device:R
- 3V3: value TestPoint -> 3V3
- OSC1: renamed from TP2; value CLKOUT -> OSC
- renumbered TP3 to GND1, TP1 to WDO1
Connections:
- net DCAN1RX: now also U3.4 (RXD)
- net DCAN1TX: now also U3.1 (TXD)
- net DGND: now also C6.2, U5.5 (GND), R12.2, R13.2; no longer D2.1 (K), D3.1 (K)
- net VDD_3V3B: no longer 3V3.1, C1.1, C10.1, C12.1, C3.1, C6.1, C8.1, D1.2, D3.2 (A), H5.37 (Pin_37), H6.27 (Pin_27), H6.28 (Pin_28), R1.2, R2.1, U1.P9_32 (VDD_ADC), U3.3 (VCC), U5.8 (VCC), U6.2 (VCC), U7.5 (~{SHUTDOWN}), U7.8 (+Vs)
- net 3V3: now reaches C2.2
- net 3V3: now also 3V3.1, C1.1, C10.1, C12.1, C3.1, C6.1, C8.1, D1.2, D3.2 (A), H5.37 (Pin_37), H6.27 (Pin_27), H6.28 (Pin_28), R1.2, R2.1, U3.3 (VCC), U4.8 (VCC), U5.8 (VCC), U6.2 (VCC), U7.5 (~{SHUTDOWN}), U7.8 (+Vs); no longer U3.1 (TXD)
- new net: D2.1 (K), R12.1
- new net: D3.1 (K), R13.1
- no-connect marks 109 -> 111
Other:
- moved on the sheet: 3V3, C10, C2
