File: flight-subsystem-designs/cdh/flight-computer/OBCV7/OBCV7.kicad_sch (KiCad schematic)
At the start: 44 parts, among them U1 BEAGLEBONEBLACK, U3 TCAN337G, U4 MCP7940N-xSN, U5 ADM3485EARZ, U6 MAX706RESA+T, U7 TMP36xS

Commit message: Technology is truley hubris manifest
Parts:
- added R10: 10k, Resistor_SMD:R_0805_2012Metric_Pad1.20x1.40mm_HandSolder, symbol Device:R
- C5: value 5nF -> 10nF
Connections:
- net ADCS_BOOT: now also H6.20 (Pin_20); no longer H6.18 (Pin_18)
- net ADCS_ENABLE: now also H6.18 (Pin_18); no longer H6.20 (Pin_20)
- net DGND: now also H6.31 (Pin_31), H6.32 (Pin_32), R10.2
- net MRV: now also U6.8 (*WDO), WDO1.1
- net at U3.8 (S): now also R10.1
- no-connect marks 111 -> 108

Commit message: watchdog corrections and other shi
Parts:
- added C13, C14: 100nf, Capacitor_SMD:C_0805_2012Metric_Pad1.18x1.45mm_HandSolder, symbol Device:C
- added S1: EG1215AA, Footprints:SW_EG1215AA, symbol EG1215AA:EG1215AA
- U6: value MAX706RESA+T -> MAX706ARESA+T
Connections:
- net 3V3: now also C14.2; no longer U6.2 (VCC)
- net DGND: now also C13.1, C14.1
- net GPIO3_20: now also S1.1; no longer U6.6 (WDI)
- net MRV: no longer U1.P9_11 (UART4_RXD)
- net VDD_3V3B: now also U6.2 (VCC), C13.2
- new net: S1.2, U6.6 (WDI)
- no-connect marks 108 -> 109
Other:
- note added: "keep near chip"
