File: flight-subsystem-designs/payload/RealQuadcellAmp/Quadcell_Rev4/Quadcell_Rev4.kicad_sch (KiCad schematic)
At the start: 52 parts, among them J1 Screw_Terminal_01x02, J2 Conn_01x04_Pin, J3 Conn_01x04_Pin, U1 OPA2192IDR, U2 OPA2192IDR, U3 OPA2192IDR, U4 OPA2192IDR, U6 LM2904

Commit message: qc
Parts:
- removed C1, C10, C4, C7: 5 pf, Capacitor_SMD:C_0805_2012Metric_Pad1.18x1.45mm_HandSolder, symbol Device:C
- removed C11, C2, C5, C8: 3 pf, Capacitor_SMD:C_0805_2012Metric_Pad1.18x1.45mm_HandSolder, symbol Device:C
- removed C12, C3, C6, C9: 330 pf, Capacitor_SMD:C_0805_2012Metric_Pad1.18x1.45mm_HandSolder, symbol Device:C
- removed R10, R14, R2, R6: 1 MΩ, Resistor_SMD:R_0805_2012Metric_Pad1.20x1.40mm_HandSolder, symbol Device:R
- removed R11, R15, R3, R7: 15 MΩ, Resistor_SMD:R_0805_2012Metric_Pad1.20x1.40mm_HandSolder, symbol Device:R
- removed R12, R16, R4, R8: 38.1 kΩ, Resistor_SMD:R_0805_2012Metric_Pad1.20x1.40mm_HandSolder, symbol Device:R
- removed R13, R5, R9: 68.1 kΩ, Resistor_SMD:R_0805_2012Metric_Pad1.20x1.40mm_HandSolder, symbol Device:R
- removed TP1, TP10, TP11, TP2, TP4, TP5, TP7, TP8: TestPoint, TestPoint:TestPoint_Pad_2.0x2.0mm, symbol Connector:TestPoint
- removed U1, U2, U3, U4: OPA2192IDR, DGK0008A_N_TEX, symbol New_Library:OPA2192IDR
- added D1: LED, Diode_SMD:D_0805_2012Metric, symbol Device:LED
- added H1, H2, H3, H4: MountingHole_Pad, MountingHole:MountingHole_3mm_Pad_Via, symbol Mechanical:MountingHole_Pad
- added J4: Conn_01x02_Pin, Connector_PinHeader_2.54mm:PinHeader_1x02_P2.54mm_Vertical, symbol Connector:Conn_01x02_Pin
- J1: footprint TerminalBlock:TerminalBlock_bornier-2_P5.08mm -> TerminalBlock_Altech:Altech_AK100_1x02_P5.00mm
- R1: value 68.1k -> 150; footprint Resistor_SMD:R_0805_2012Metric_Pad1.20x1.40mm_HandSolder -> Resistor_SMD:R_0805_2012Metric
- R31, R33: footprint Resistor_SMD:R_0805_2012Metric_Pad1.20x1.40mm_HandSolder -> Resistor_SMD:R_0805_2012Metric
- TP_+BATT1, TP_GND1, TP_QUADGND1: footprint TestPoint:TestPoint_THTPad_1.0x1.0mm_Drill0.5mm -> TestPoint:TestPoint_Loop_D2.50mm_Drill1.0mm
- U5: footprint OSI:InGaAS-Q1000 -> Quadcell_Components:InGaAS-Q1000
Connections:
- net GND: now also R1.2
- net QUAD_GND: now also H1.1, H2.1, H3.1, H4.1
- net VCC: now also D1.2 (A)
- net OUT1: no longer names the net of R1.1
- net OUT1: now also D1.1 (K)
- net OUT5 renamed STAGE2_OUT1
- net OUT6 renamed STAGE2_OUT2
- net OUT7 renamed STAGE2_OUT3
- net OUT8 renamed STAGE2_OUT4
- new net I2C_SCL: J4.2 (Pin_2)
- new net I2C_SDA: J4.1 (Pin_1)
Other:
- added sheet amplification (amplification.kicad_sch)
- added sheet digital_conversion (digital_conversion.kicad_sch)
- note removed: "stage one"
- note removed: "stage two"
- moved on the sheet: C13, C14, J1, J2, J3, R31, R33, TP_+BATT1, TP_GND1, TP_QUADGND1, U5, U6A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
