File: flight-subsystem-designs/power/power-distribution/PowerDistribution.kicad_pcb (KiCad board)
At the start: 4 copper layers, 90.2 x 96 mm, 142 parts, among them J1 Conn_02x26_Odd_Even, J11 Conn_01x04, J12 Conn_01x04, J13 Conn_01x04, J15 Conn_01x02, J2 Conn_02x26_Odd_Even, J3 Conn_01x02, J4 Conn_01x02, J5 Conn_01x02, J6 Conn_01x02, J8 Conn_01x02, Q1 BC848ALT1G, Q2 IRLML2803PBFCT, Q3 IRLML2803PBFCT, Q4 NMOS, Q5 NMOS, U1 LT8610, U12 LTM8062AIV-PBF, U16 INA219AxD, U17 INA219AxD, U18 INA219AxD, U2 LT8610, U21 INA219AxD, U6 LT8610

Commit message: feat: pdu 4.0 in progress
Parts:
- added R36: TBD, Resistor_SMD:R_0603_1608Metric, F.Cu at (260.7, 76.0)
- added R39: 50k, Resistor_SMD:R_0603_1608Metric, F.Cu at (260.7, 73.5)
- C35: renamed from C3; footprint Capacitor_SMD:C_0805_2012Metric -> Capacitor_SMD:C_1206_3216Metric
- C36: renamed from C12; footprint Capacitor_SMD:C_0805_2012Metric -> Capacitor_SMD:C_1206_3216Metric
- R10: renamed from R52; value 2m -> 40m
- R11: renamed from R43; value 2m -> 40m
- R3: renamed from R33; value 2m -> 10m
- R31: renamed from R11; footprint Resistor_SMD:R_0603_1608Metric -> Capacitor_SMD:C_1206_3216Metric
- R9: renamed from R55; value 2m -> 40m
- renumbered C15 to C1, C45 to C10, C47 to C11, C4 to C12, C7 to C13, C19 to C14, C1 to C15, C20 to C16, C8 to C17, C29 to C18, C13 to C19, C27 to C2, C17 to C20, C25 to C21, C5 to C22, C9 to C23, C21 to C24, C2 to C25, C10 to C26, C22 to C27, C30 to C28, C14 to C29, C42 to C3, C18 to C30, C26 to C31, C23 to C32, C6 to C33, C11 to C34, C24 to C37, C34 to C38, C35 to C39, C51 to C4, C33 to C5, C32 to C6, C31 to C7, C50 to C8, C46 to C9, D9 to D1, D1 to D10, D7 to D11, D11 to D12, D8 to D2, D10 to D3, D13 to D4, D4 to D5, D5 to D6, D6 to D7, D2 to D8, D3 to D9, J15 to J1, J13 to J10, J5 to J11, J8 to J12, J1 to J2, J6 to J5, J2 to J7, J11 to J8, J12 to J9, L4 to L1, L1 to L2, L2 to L3, L3 to L4, Q4 to Q1, Q5 to Q2, Q1 to Q3, Q2 to Q4, Q3 to Q5, R15 to R1, R35 to R12, R37 to R13, R39 to R14, R2 to R15, R5 to R16, R7 to R17, R4 to R18, R6 to R19, R18 to R2, R9 to R20, R1 to R21, R3 to R22, R8 to R23, R10 to R24, R30 to R25, R14 to R26, R12 to R29, R13 to R30, R20 to R32, R19 to R33, R22 to R34, R23 to R35, R21 to R37, R24 to R38, R59 to R4, R25 to R40, R26 to R41, R34 to R42, R40 to R43, R31 to R44, R16 to R45, R17 to R46, R57 to R5, R32 to R6, R36 to R7, R38 to R8, TP3 to TP1, TP1 to TP3, U4 to U1, U3 to U10, U9 to U11, U10 to U12, U5 to U13, U12 to U14, U13 to U15, U11 to U16, U7 to U17, U8 to U18, U21 to U2, U17 to U3, U16 to U4, U18 to U5, U1 to U6, U2 to U7, U6 to U8, U14 to U9
Connections:
- net /CHARGE_VIN renamed Net-(C38-Pad2)
- net /CHRG renamed /~{CHRG_STAT}
- net /FAULT renamed /~{CHRG_FAULT}
- net Net-(U11-VOUT-Pad3) renamed /ADCS_PWR
- J10 pad 1: /SOLAR_IN_-Y -> GND
- J10 pad 2: 3V3 -> /SOLAR_IN_-Y
- J10 pad 3: /SOLAR_TMP_-Y -> /SOLAR_IN_-Y
- J2 pad 48: /SOLAR_TMP_+Y -> unconnected-(J2-Pin_48-Pad48)
- J2 pad 49: /SOLAR_TMP_-Z -> unconnected-(J2-Pin_49-Pad49)
- J2 pad 50: /SOLAR_TMP_-Y -> unconnected-(J2-Pin_50-Pad50)
- J3 pad 2: /SOLAR_PRE_MPPT -> VINA
- J8 pad 1: /SOLAR_IN_-Z -> GND
- J8 pad 2: 3V3 -> /SOLAR_IN_-Z
- J8 pad 3: /SOLAR_TMP_-Z -> /SOLAR_IN_-Z
- J9 pad 1: /SOLAR_IN_+Y -> GND
- J9 pad 2: 3V3 -> /SOLAR_IN_+Y
- J9 pad 3: /SOLAR_TMP_+Y -> /SOLAR_IN_+Y
- U14 pad B4: GND -> (no net)
- U14 pad B6: VBATT -> GND
- U14 pad E1: GND -> (no net)
- U14 pad E2: GND -> (no net)
- U14 pad E3: GND -> (no net)
- U14 pad E4: GND -> (no net)
- U14 pad E5: GND -> (no net)
- U14 pad K4: /SOLAR_PRE_MPPT -> VINA
- U14 pad K5: /SOLAR_PRE_MPPT -> VINA
- U14 pad K6: /SOLAR_PRE_MPPT -> VINA
- U14 pad L4: /SOLAR_PRE_MPPT -> VINA
- U14 pad L5: /SOLAR_PRE_MPPT -> VINA
- U14 pad L6: /VIN_REG -> VINA
- U16 pad 1: unconnected-(U11-ILIM-Pad1) -> Net-(U16-ILIM)
- U16 pad 10: VS -> VBATT
- U16 pad 11: VS -> VBATT
- U16 pad 12: VS -> VBATT
- U16 pad 13: VS -> VBATT
- U16 pad 15: unconnected-(U11-EN-Pad15) -> /ADCS_PWR_EN
- U16 pad 16: unconnected-(U11-DIAG_EN-Pad16) -> /ADCS_PWR_DIAG
- U16 pad 17: unconnected-(U11-FAULT-Pad17) -> /~{ADCS_PWR_FAULT}
- U16 pad 18: unconnected-(U11-GND-Pad18) -> GND
- U16 pad 20: unconnected-(U11-SNS-Pad20) -> /ADCS_PWR_SNS
Routing:
- net (no net): track 0.00 -> 39.9 mm
- net /SOLAR_IN_+Y: track 3.76 -> 42.0 mm, vias 0 -> 3
- net /SOLAR_TMP_+Y: track 35.3 -> 0.00 mm, vias 2 -> 0
- net /SOLAR_TMP_-Y: track 29.5 -> 0.00 mm
- net /SOLAR_TMP_-Z: track 10.3 -> 0.00 mm
- net 3V3: track 81.2 -> 71.4 mm, vias 12 -> 9
- net /SOLAR_IN_-Z: track 3.89 -> 8.26 mm, vias 0 -> 1
- net /SOLAR_IN_-Y: track 3.72 -> 6.23 mm, vias 0 -> 1
- net VINA: vias 0 -> 4
- net /SOLAR_PRE_MPPT: vias 4 -> 0
- added copper zone on B.Cu, net VINA
- added copper zone on F.Cu, net VINA
- removed copper zone on B.Cu, net /SOLAR_PRE_MPPT
- removed copper zone on F.Cu, net /SOLAR_PRE_MPPT
- removed copper zone on F.Cu, net /VIN_REG

Commit message: updates from old computer
Parts:
- added J1: Conn_02x07_Top_Bottom, Connector_Harwin:Harwin_LTek-Male_2x07_P2.00mm_Vertical_StrainRelief, F.Cu at (267.8, 81.6)
- added U19: STM32L431CBTx, Package_QFP:LQFP-48_7x7mm_P0.5mm, F.Cu at (268.8, 125.2)
Connections:
- J2 pad 10: GND_REF -> unconnected-(J2-Pin_10-Pad10)
- J2 pad 11: GND_REF -> unconnected-(J2-Pin_11-Pad11)
- J2 pad 12: GND_REF -> unconnected-(J2-Pin_12-Pad12)
- J2 pad 37: KAPTON_EN -> /KAPTON_EN
- J2 pad 9: GND_REF -> unconnected-(J2-Pin_9-Pad9)
- U14 pad B6: GND -> VBATT

Commit message: Chris' laser driver files
Parts:
- removed C20: 0.1uF, Capacitor_SMD:C_0603_1608Metric
- removed C30: 1uF, Capacitor_SMD:C_0603_1608Metric
- removed D6: 150060AS75000, LED_SMD:LED_0603_1608Metric
- removed the J1 at (177.6, 123.2)
- removed J5: Conn_01x02, Connector_Molex:Molex_Pico-Lock_205338-0002_1x02-1MP_P2.00mm_Horizontal
- removed R27: 150, Resistor_SMD:R_0603_1608Metric
- removed R36: TBD, Resistor_SMD:R_0603_1608Metric
- removed R39: 50k, Resistor_SMD:R_0603_1608Metric
- removed the R41 at (211.4, 73.6)
- removed U11: ~, Package_SO:SOIC-8_3.9x4.9mm_P1.27mm
- removed U16: ~, Package_DFN_QFN:Texas_RGW0020A_VQFN-20-1EP_5x5mm_P0.65mm_EP3.15x3.15mm_ThermalVias
Routing:
- net KAPTON_EN: track 79.0 -> 0.00 mm
- net /KAPTON_EN: track 0.00 -> 79.0 mm
- net (no net): track 39.9 -> 87.3 mm, vias 0 -> 6
- net KAPTON_PWR: track 45.1 -> 0.00 mm, vias 5 -> 0
- net Net-(D6-K): track 2.37 -> 0.00 mm, vias 1 -> 0
- added copper zone on In2.Cu, net (none)
- removed copper zone on In2.Cu, net KAPTON_PWR

Commit message: feat: PDU updates and laser driver v1.0.1
Connections:
- C22 pad 2: EDFA_5V -> /EDFA_5V
- C35 pad 2: EDFA_5V -> /EDFA_5V
- D8 pad 2: EDFA_5V -> /EDFA_5V
- J2 pad 31: 5V_S_EN -> /5V_S_EN
- J2 pad 39: 3V3_S_EN -> /3V3_S_EN
- J2 pad 40: EDFA_5V_EN -> /EDFA_5V_EN
- J2 pad 42: EDFA_5V_S -> /EDFA_5V_S
- J2 pad 44: EDFA_5V_S -> /EDFA_5V_S
- J2 pad 45: 5V_S -> /5V_S
- J2 pad 46: 5V_S -> /5V_S
- L2 pad 2: EDFA_5V -> /EDFA_5V
- R21 pad 1: EDFA_5V -> /EDFA_5V
- R22 pad 2: EDFA_5V -> /EDFA_5V
- TP1 pad 1: EDFA_5V -> /EDFA_5V
- U6 pad 14: EDFA_5V -> /EDFA_5V
Routing:
- net /EDFA_5V: track 0.00 -> 7.13 mm, vias 0 -> 3
- net EDFA_5V: track 36.9 -> 29.8 mm, vias 8 -> 5
Changed lines of the file:
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@@
 	(net 222 "unconnected-(J2-Pin_10-Pad10)")
 	(net 223 "unconnected-(J2-Pin_9-Pad9)")
+	(net 224 "/EDFA_5V")
+	(net 225 "/3V3_S_EN")
+	(net 226 "/EDFA_5V_EN")
+	(net 227 "/5V_S")
+	(net 228 "/EDFA_5V_S")
+	(net 229 "/5V_S_EN")
 	(footprint "Capacitor_SMD:C_0805_2012Metric"
 		(layer "F.Cu")
@@
 		)
 		(property ki_fp_filters "CP_*")
-		(sheetname "/")
-		(sheetfile "PowerDistribution.kicad_sch")
+		(sheetname "/Switches/")
+		(sheetfile "switches.kicad_sch")
 		(attr smd)
 		(fp_line
@@
 		)
 		(property ki_fp_filters "CP_*")
-		(sheetname "/")
-		(sheetfile "PowerDistribution.kicad_sch")
+		(sheetname "/Switches/")
+		(sheetfile "switches.kicad_sch")
 		(attr smd)
 		(fp_line
@@
 			(layers "F.Cu" "F.Mask" "F.Paste")
 			(roundrect_rratio 0.25)
-			(net 5 "EDFA_5V")
+			(net 224 "/EDFA_5V")
 			(pintype "passive")
 		)
@@
 		)
 		(property ki_fp_filters "C_*")
-		(sheetname "/")
-		(sheetfile "PowerDistribution.kicad_sch")
+		(sheetname "/Switches/")
+		(sheetfile "switches.kicad_sch")
 		(attr smd)
 		(fp_line
@@
 		)
 		(property ki_fp_filters "LED* LED_SMD:* LED_THT:*")
-		(sheetname "/")
-		(sheetfile "PowerDistribution.kicad_sch")
+		(sheetname "/Switches/")
+		(sheetfile "switches.kicad_sch")
 		(attr smd)
 		(fp_line
@@
 			)
 		)
-		(sheetname "/")
-		(sheetfile "PowerDistribution.kicad_sch")
+		(sheetname "/Switches/")
+		(sheetfile "switches.kicad_sch")
 		(attr smd)
 		(fp_line
@@
 		)
 		(property ki_fp_filters "C_*")
-		(sheetname "/")
-		(sheetfile "PowerDistribution.kicad_sch")
+		(sheetname "/Switches/")
+		(sheetfile "switches.kicad_sch")
 		(attr smd)
 		(fp_line
@@
 			(layers "F.Cu" "F.Mask" "F.Paste")
 			(roundrect_rratio 0.25)
-			(net 5 "EDFA_5V")
+			(net 224 "/EDFA_5V")
 			(pinfunction "A")
 			(pintype "passive")
@@
 		)
 		(property ki_fp_filters "C_*")
-		(sheetname "/")
-		(sheetfile "PowerDistribution.kicad_sch")
+		(sheetname "/Switches/")
+		(sheetfile "switches.kicad_sch")
 		(attr smd)
 		(fp_line
@@
 			(layers "F.Cu" "F.Mask" "F.Paste")
 			(roundrect_rratio 0.243902)
-			(net 5 "EDFA_5V")
+			(net 224 "/EDFA_5V")
 			(pintype "passive")
 		)
@@
 			)
 		)
-		(sheetname "/")
-		(sheetfile "PowerDistribution.kicad_sch")
+		(sheetname "/Switches/")
+		(sheetfile "switches.kicad_sch")
 		(attr smd)
 		(fp_line
@@
 			(layers "F.Cu" "F.Mask" "F.Paste")
 			(roundrect_rratio 0.25)
-			(net 5 "EDFA_5V")
+			(net 224 "/EDFA_5V")
 			(pinfunction "BIAS")
 			(pintype "input")
@@
 			)
 		)
-		(sheetname "/")
-		(sheetfile "PowerDistribution.kicad_sch")
+		(sheetname "/Switches/")
+		(sheetfile "switches.kicad_sch")
 		(attr smd)
 		(fp_line
@@
 			(layers "*.Cu" "*.Mask")
 			(remove_unused_layers no)
-			(net 132 "5V_S_EN")
+			(net 229 "/5V_S_EN")
 			(pinfunction "Pin_31")
 			(pintype "passive")
@@
 			(layers "*.Cu" "*.Mask")
 			(remove_unused_layers no)
-			(net 133 "3V3_S_EN")
+			(net 225 "/3V3_S_EN")
 			(pinfunction "Pin_39")
 			(pintype "passive")
@@
 			(layers "*.Cu" "*.Mask")
 			(remove_unused_layers no)
-			(net 130 "EDFA_5V_EN")
+			(net 226 "/EDFA_5V_EN")
 			(pinfunction "Pin_40")
 			(pintype "passive")
@@
 			(layers "*.Cu" "*.Mask")
 			(remove_unused_layers no)
-			(net 44 "EDFA_5V_S")
+			(net 228 "/EDFA_5V_S")
 			(pinfunction "Pin_42")
 			(pintype "passive")
@@
 			(layers "*.Cu" "*.Mask")
 			(remove_unused_layers no)
-			(net 44 "EDFA_5V_S")
+			(net 228 "/EDFA_5V_S")
 			(pinfunction "Pin_44")
 			(pintype "passive")
@@
 			(layers "*.Cu" "*.Mask")
 			(remove_unused_layers no)
-			(net 49 "5V_S")
+			(net 227 "/5V_S")
 			(pinfunction "Pin_45")
 			(pintype "passive")
@@
 			(layers "*.Cu" "*.Mask")
 			(remove_unused_layers no)
-			(net 49 "5V_S")
+			(net 227 "/5V_S")
 			(pinfunction "Pin_46")
 			(pintype "passive")
@@
 			(layers "F.Cu" "F.Mask" "F.Paste")
 			(roundrect_rratio 0.217391)
-			(net 5 "EDFA_5V")
+			(net 224 "/EDFA_5V")
 			(pintype "passive")
 		)
@@
 			(layers "*.Cu" "*.Mask")
 			(remove_unused_layers no)
-			(net 5 "EDFA_5V")
+			(net 224 "/EDFA_5V")
 			(pinfunction "1")
 			(pintype "passive")
@@
 		)
 		(property ki_fp_filters "LED* LED_SMD:* LED_THT:*")
-		(sheetname "/")
-		(sheetfile "PowerDistribution.kicad_sch")
+		(sheetname "/Switches/")
+		(sheetfile "switches.kicad_sch")
 		(attr smd)
 		(fp_line
@@
 			(size 0.98 3.4)
 			(layers "F.Cu" "F.Mask" "F.Paste")
-			(net 5 "EDFA_5V")
+			(net 224 "/EDFA_5V")
 			(pinfunction "2")
 			(pintype "passive")
@@
 		)
 		(property ki_fp_filters "CP_*")
-		(sheetname "/")
-		(sheetfile "PowerDistribution.kicad_sch")
+		(sheetname "/Switches/")
+		(sheetfile "switches.kicad_sch")
 		(attr smd)
 		(fp_line
@@
 		)
 		(property ki_fp_filters "LED* LED_SMD:* LED_THT:*")
-		(sheetname "/")
-		(sheetfile "PowerDistribution.kicad_sch")
+		(sheetname "/Switches/")
+		(sheetfile "switches.kicad_sch")
 		(attr smd)
 		(fp_line
@@
 		)
 		(property ki_fp_filters "R_*")
-		(sheetname "/")
-		(sheetfile "PowerDistribution.kicad_sch")
+		(sheetname "/Switches/")
+		(sheetfile "switches.kicad_sch")
 		(attr smd)
 		(fp_line
@@
 		)
 		(property ki_fp_filters "R_*")
-		(sheetname "/")
-		(sheetfile "PowerDistribution.kicad_sch")
+		(sheetname "/Switches/")
+		(sheetfile "switches.kicad_sch")
 		(attr smd)
 		(fp_line
@@
 			(layers "B.Cu" "B.Mask" "B.Paste")
 			(roundrect_rratio 0.25)
-			(net 5 "EDFA_5V")
+			(net 224 "/EDFA_5V")
 			(pintype "passive")
 		)
@@
 		)
 		(property ki_fp_filters "R_*")
-		(sheetname "/")
-		(sheetfile "PowerDistribution.kicad_sch")
+		(sheetname "/Switches/")
+		(sheetfile "switches.kicad_sch")
 		(attr smd)
 		(fp_line
@@
 	)
 	(segment
-		(start 201.367303 119.969423)
-		(end 201.835954 120.438074)
-		(width 0.7)
-		(layer "F.Cu")
-		(net 5)
-	)
-	(segment
 		(start 235.487537 110.811117)
 		(end 236.576009 111.899589)
@@
 	)
 	(segment
-		(start 198.265904 119.969423)
-		(end 201.367303 119.969423)
-		(width 0.7)
-		(layer "F.Cu")
-		(net 5)
-	)
-	(segment
 		(start 250.7995 110.035556)
 		(end 242.050688 110.035556)
@@
 	)
 	(segment
-		(start 197.4833 124.44)
-		(end 197.739671 124.183629)
-		(width 0.3)
-		(layer "F.Cu")
-		(net 5)
-	)
-	(segment
 		(start 242.050688 110.035556)
 		(end 240.005127 112.081117)
@@
 	)
 	(segment
-		(start 196.235 124.44)
-		(end 197.4833 124.44)
-		(width 0.3)
-		(layer "F.Cu")
-		(net 5)
-	)
-	(segment
 		(start 229.503855 110.811117)
 		(end 234.453855 110.811117)
@@
 	)
 	(via
-		(at 201.835954 121.581074)
-		(size 0.6)
-		(drill 0.25)
-		(layers "F.Cu" "B.Cu")
-		(net 5)
-	)
-	(via
 		(at 239.090855 112.081117)
 		(size 0.7)
@@
 		(net 5)
 	)
-	(via
-		(at 201.835954 120.438074)
-		(size 0.6)
-		(drill 0.25)
-		(layers "F.Cu" "B.Cu")
-		(net 5)
-	)
-	(via
-		(at 197.739671 124.183629)
-		(size 0.6)
-		(drill 0.25)
-		(layers "F.Cu" "B.Cu")
-		(net 5)
-	)
-	(segment
-		(start 200.749162 122.667866)
-		(end 200.53378 122.667866)
-		(width 0.3)
-		(layer "B.Cu")
-		(net 5)
-	)
-	(segment
-		(start 201.835954 121.581074)
-		(end 200.749162 122.667866)
-		(width 0.3)
-		(layer "B.Cu")
-		(net 5)
-	)
 	(segment
 		(start 192.281294 76.437372)
@@
 		(net 220)
 	)
+	(segment
+		(start 201.367303 119.969423)
+		(end 201.835954 120.438074)
+		(width 0.7)
+		(layer "F.Cu")
+		(net 224)
+	)
+	(segment
+		(start 198.265904 119.969423)
+		(end 201.367303 119.969423)
+		(width 0.7)
+		(layer "F.Cu")
+		(net 224)
+	)
+	(segment
+		(start 197.4833 124.44)
+		(end 197.739671 124.183629)
+		(width 0.3)
+		(layer "F.Cu")
+		(net 224)
+	)
+	(segment
+		(start 196.235 124.44)
+		(end 197.4833 124.44)
+		(width 0.3)
+		(layer "F.Cu")
+		(net 224)
+	)
+	(via
+		(at 201.835954 121.581074)
+		(size 0.6)
+		(drill 0.25)
+		(layers "F.Cu" "B.Cu")
+		(net 224)
+	)
+	(via
+		(at 201.835954 120.438074)
+		(size 0.6)
+		(drill 0.25)
+		(layers "F.Cu" "B.Cu")
+		(net 224)
+	)
+	(via
+		(at 197.739671 124.183629)
+		(size 0.6)
+		(drill 0.25)
+		(layers "F.Cu" "B.Cu")
+		(net 224)
+	)
+	(segment
+		(start 200.749162 122.667866)
+		(end 200.53378 122.667866)
+		(width 0.3)
+		(layer "B.Cu")
+		(net 224)
+	)
+	(segment
+		(start 201.835954 121.581074)
+		(end 200.749162 122.667866)
+		(width 0.3)
+		(layer "B.Cu")
+		(net 224)
+	)
 	(zone

Commit message: feat: PDU 4.0.0 (WIP)
Parts:
- removed C39: 4.7uF, Capacitor_Tantalum_SMD:CP_EIA-3528-12_Kemet-T
- removed R44: 549k, Resistor_SMD:R_0603_1608Metric
- added C20: 10uF, Capacitor_SMD:C_0603_1608Metric, F.Cu at (112.2, 56.0)
- added C30: 0.1uF, Capacitor_SMD:C_0603_1608Metric, F.Cu at (112.2, 58.5)
- added C40: 0.1uF, Capacitor_SMD:C_0603_1608Metric, F.Cu at (112.2, 61.0)
- added C41: 0.1uF, Capacitor_SMD:C_0603_1608Metric, F.Cu at (112.2, 63.5)
- added C42: 0.1uF, Capacitor_SMD:C_0603_1608Metric, F.Cu at (112.2, 66.0)
- added C43: 10nF, Capacitor_SMD:C_0603_1608Metric, F.Cu at (112.2, 68.5)
- added C44: 1uF, Capacitor_SMD:C_0603_1608Metric, F.Cu at (116.3, 56.0)
- added C45: 1uF, Capacitor_SMD:C_0603_1608Metric, F.Cu at (116.3, 58.5)
- added C46: 0.1uF, Capacitor_SMD:C_0603_1608Metric, F.Cu at (85.7, 85.8)
- added C47: 10pF, Capacitor_SMD:C_0603_1608Metric, F.Cu at (94.7, 76.5)
- added C48: 10pF, Capacitor_SMD:C_0603_1608Metric, F.Cu at (94.7, 79.0)
- added C49: 1uF, Capacitor_SMD:C_0603_1608Metric, F.Cu at (82.5, 96.0)
- added C50: 1uF, Capacitor_SMD:C_0603_1608Metric, F.Cu at (133.8, 44.6)
- added C51: 0.01uF, Capacitor_SMD:C_0603_1608Metric, F.Cu at (133.8, 47.2)
- added C52: 10uF, Capacitor_SMD:C_0603_1608Metric, F.Cu at (133.8, 49.7)
- added C53: 0.1uF, Capacitor_SMD:C_0603_1608Metric, F.Cu at (119.0, 83.0)
- added C54: 22uF, Capacitor_SMD:C_0805_2012Metric, F.Cu at (307.7, 60.8)
- added C55: 0.1uF, Capacitor_SMD:C_0805_2012Metric, F.Cu at (307.7, 63.8)
- added C56: 4.7uF, Capacitor_Tantalum_SMD:CP_EIA-3528-12_Kemet-T, F.Cu at (132.0, 96.2)
- added D13: GREEN, LED_SMD:LED_0603_1608Metric, F.Cu at (116.6, 132.6)
- added D14: PINK, LED_SMD:LED_0603_1608Metric, F.Cu at (116.6, 128.0)
- added D15: PINK, LED_SMD:LED_0603_1608Metric, F.Cu at (110.5, 128.0)
- added D16: PINK, LED_SMD:LED_0603_1608Metric, F.Cu at (110.5, 130.6)
- added D17: PINK, LED_SMD:LED_0603_1608Metric, F.Cu at (110.5, 133.2)
- added D18: RED, LED_SMD:LED_0603_1608Metric, F.Cu at (110.5, 135.8)
- added D19: RED, LED_SMD:LED_0603_1608Metric, F.Cu at (312.9, 51.3)
- added D6: AMBER, LED_SMD:LED_0603_1608Metric, F.Cu at (126.5, 46.5)
- added FB1: 120R, Inductor_SMD:L_0805_2012Metric, F.Cu at (111.5, 74.1)
- added J14: Molex 205338-2, Connector_Molex:Molex_Pico-Lock_205338-0002_1x02-1MP_P2.00mm_Horizontal, F.Cu at (297.0, 132.5)
- added J15: Battery Header, Connector_PinHeader_2.54mm:PinHeader_2x08_P2.54mm_Vertical, F.Cu at (151.0, 92.5)
- added J5: Molex 205338-2, Connector_Molex:Molex_Pico-Lock_205338-0002_1x02-1MP_P2.00mm_Horizontal, F.Cu at (281.1, 111.4)
- added J6: Molex 205338-2, Connector_Molex:Molex_Pico-Lock_205338-0002_1x02-1MP_P2.00mm_Horizontal, F.Cu at (297.0, 122.2)
- added JP1: Jumper_2_Open, Jumper:SolderJumper-2_P1.3mm_Open_TrianglePad1.0x1.5mm, F.Cu at (299.3, 51.8)
- added JP2: Jumper_2_Open, Jumper:SolderJumper-2_P1.3mm_Open_TrianglePad1.0x1.5mm, F.Cu at (299.3, 55.3)
- added JP3: Jumper_2_Open, Jumper:SolderJumper-2_P1.3mm_Open_TrianglePad1.0x1.5mm, F.Cu at (299.3, 58.9)
- added JP4: Jumper_2_Open, Jumper:SolderJumper-2_P1.3mm_Open_TrianglePad1.0x1.5mm, F.Cu at (299.3, 62.4)
- added JP5: Jumper_2_Open, Jumper:SolderJumper-2_P1.3mm_Open_TrianglePad1.0x1.5mm, F.Cu at (299.3, 66.0)
- added L5: AIMC-0805-2N2S-T, Inductor_SMD:L_0805_2012Metric, F.Cu at (312.2, 60.7)
- added Q6: NMOS, Package_TO_SOT_SMD:TSOT-23, F.Cu at (308.2, 52.4)
- added Q7: NMOS, Package_TO_SOT_SMD:TSOT-23, F.Cu at (308.2, 57.1)
- added R27: 150, Resistor_SMD:R_0603_1608Metric, F.Cu at (290.7, 107.5)
- added R36: 10k, Resistor_SMD:R_0603_1608Metric, F.Cu at (101.3, 50.8)
- added R39: 150, Resistor_SMD:R_0603_1608Metric, F.Cu at (133.8, 52.2)
- added R47: 150, Resistor_SMD:R_0603_1608Metric, F.Cu at (288.8, 61.3)
- added R48: 150, Resistor_SMD:R_0603_1608Metric, F.Cu at (303.5, 51.2)
- added R49: 150, Resistor_SMD:R_0603_1608Metric, F.Cu at (303.5, 53.8)
- added R50: 150, Resistor_SMD:R_0603_1608Metric, F.Cu at (303.5, 56.3)
- added R51: 10k, Resistor_SMD:R_0603_1608Metric, F.Cu at (119.0, 85.5)
- added R52: 10k, Resistor_SMD:R_0603_1608Metric, F.Cu at (119.0, 88.0)
- added R53: 150, Resistor_SMD:R_0603_1608Metric, F.Cu at (311.2, 71.0)
- added R54: 1M, Resistor_SMD:R_0603_1608Metric, F.Cu at (303.5, 58.8)
- added R55: 1M, Resistor_SMD:R_0603_1608Metric, F.Cu at (303.5, 61.3)
- added R56: 150, Resistor_SMD:R_0603_1608Metric, F.Cu at (303.5, 63.8)
- added R57: 10k, Resistor_SMD:R_0603_1608Metric, F.Cu at (288.8, 63.8)
- added R58: 10k, Resistor_SMD:R_0603_1608Metric, F.Cu at (288.8, 66.3)
- added R59: 10k, Resistor_SMD:R_0603_1608Metric, F.Cu at (288.8, 68.8)
- added R60: 10k, Resistor_SMD:R_0603_1608Metric, F.Cu at (299.2, 71.0)
- added R61: 10k, Resistor_SMD:R_0603_1608Metric, F.Cu at (299.2, 73.5)
- added R62: 10k, Resistor_SMD:R_0603_1608Metric, F.Cu at (299.2, 76.0)
- added R63: 150, Resistor_SMD:R_0603_1608Metric, F.Cu at (303.5, 66.3)
- added SW1: SW_Push, Button_Switch_SMD:SW_SPST_B3U-1000P, F.Cu at (81.7, 79.8)
- added TP4: LDO, TestPoint:TestPoint_Keystone_5000-5004_Miniature, F.Cu at (138.0, 45.6)
- added TP5: VBATT, TestPoint:TestPoint_Keystone_5000-5004_Miniature, F.Cu at (293.0, 56.5)
- added TP6: GND, TestPoint:TestPoint_Keystone_5000-5004_Miniature, F.Cu at (312.1, 64.2)
- added TP7: VSOLAR, TestPoint:TestPoint_Keystone_5000-5004_Miniature, F.Cu at (315.2, 66.5)
- added U11: MAX706RESA, Package_SO:SOIC-8_3.9x4.9mm_P1.27mm, F.Cu at (76.3, 71.4)
- added U16: TCAN337G, Package_SO:SOIC-8_3.9x4.9mm_P1.27mm, F.Cu at (122.0, 67.1)
- added U20: LT1761-3.3, Package_TO_SOT_SMD:TSOT-23-5, F.Cu at (121.4, 58.5)
- added Y1: 16 MHz, Crystal:Crystal_SMD_3225-4Pin_3.2x2.5mm, F.Cu at (102.8, 79.9)
- C37: footprint Capacitor_SMD:C_0805_2012Metric -> Capacitor_SMD:C_1206_3216Metric
- D10, D8, D9: value 150060VS75000 -> AMBER
- D11: value 150060VS75000 -> GREEN
- D12: value 150060VS75000 -> RED
- D4, D5, D7: value 150060AS75000 -> GREEN
- J1: value Conn_02x07_Top_Bottom -> Conn_01x05; footprint Connector_Harwin:Harwin_LTek-Male_2x07_P2.00mm_Vertical_StrainRelief -> Connector_PinHeader_2.54mm:PinHeader_1x05_P2.54mm_Vertical
- J10, J8, J9: value Conn_01x04 -> Molex 205338-4
- J3, J4: value Conn_01x02 -> Molex 205338-2
- R21: value 100k -> 10k; moved to F.Cu
- R25: value 65 -> 150
- R26: value 150 -> 642k; moved to F.Cu
- R28: value 150 -> 412k; moved to F.Cu
- R30: value 65 -> 10k; moved to F.Cu
- R31: footprint Capacitor_SMD:C_1206_3216Metric -> Resistor_SMD:R_0603_1608Metric
- R42: value 549k -> 150
- R43: value 459k -> 150
- TP1: value ~ -> EDFA
- TP2: value ~ -> 3V3
- TP3: value ~ -> 5V
- U1: value ~ -> TMP36FSZ
- U10, U12, U9: value ~ -> LTC1477CS8
- U13: value ~ -> SI4835DDY
- U15: value ~ -> MR25H256ACDF
- U17, U18: value ~ -> SI3407DV
- U19: value STM32L431CBTx -> STM32L431CBT6
- U2, U3, U4, U5: value INA219AxD -> INA219AIDR
- moved J1 182.8 mm to (86.2, 60.1)
- moved U19 177.3 mm to (102.6, 63.5)
- moved U15 167.1 mm to (94.7, 87.2)
- moved R30 161.2 mm to (101.3, 48.2)
- moved R28 122.4 mm to (131.0, 102.2)
- moved R26 122.3 mm to (131.0, 99.7)
- moved R21 119.6 mm to (82.5, 98.5), turned to 0 degrees
Connections:
- net /CS_SOL1_VIN+ renamed /Connectors/CS_SOL1_VIN+
- net /CS_SOL1_VIN- renamed /Connectors/CS_SOL1_VIN-
- net /CS_SOL2_VIN+ renamed /Connectors/CS_SOL2_VIN+
- net /CS_SOL2_VIN- renamed /Connectors/CS_SOL2_VIN-
- net /CS_SOL3_VIN+ renamed /Connectors/CS_SOL3_VIN+
- net /CS_SOL3_VIN- renamed /Connectors/CS_SOL3_VIN-
- net /FB_1 renamed /Regulators/FB_1
- net /FB_2 renamed /Regulators/FB_2
- net /FB_3 renamed /Regulators/FB_3
- net /RBF_SW renamed Net-(J6-Pin_1)
- net /SOLAR_IN_+Y renamed /Connectors/SOLAR_IN_+Y
- net /SOLAR_IN_-Y renamed /Connectors/SOLAR_IN_-Y
- net /SOLAR_IN_-Z renamed /Connectors/SOLAR_IN_-Z
- net /SW_1 renamed /Regulators/SW_1
- net /SW_2 renamed /Regulators/SW_2
- net /SW_3 renamed /Regulators/SW_3
- net /b1 renamed /Deployment/b1
- net /b2 renamed /Deployment/b2
- net /sol_1_diode renamed /Connectors/sol_1_diode
- net /sol_2_diode renamed /Connectors/sol_2_diode
- net /sol_3_diode renamed /Connectors/sol_3_diode
- C10 pad 2: 3V3_S -> 3V3
- C11 pad 2: 3V3_S -> 3V3
- C19 pad 1: EDFA_5V -> 5V
- C2 pad 2: /VBATT_IN -> /Connectors/VBATT_IN
- C22 pad 2: /EDFA_5V -> EDFA_5V
- C28 pad 2: GND -> Net-(D4-K)
- C29 pad 1: EDFA_5V_S -> 5V_2_S
- C29 pad 2: GND -> Net-(D5-K)
- C3 pad 2: /VBATT_IN -> /Connectors/VBATT_IN
- C31 pad 1: 5V_S -> 5V_1_S
- C31 pad 2: GND -> Net-(D7-K)
- C35 pad 2: /EDFA_5V -> EDFA_5V
- C8 pad 2: 3V3_S -> 3V3
- C9 pad 2: 3V3_S -> 3V3
- D1 pad 1: SOLAR_PRE_INH -> /Connectors/VSOLAR_IN
- D11 pad 2: /~{CHRG_STAT} -> /Charging/~{CHRG_STAT}
- D12 pad 2: /~{CHRG_FAULT} -> /Charging/~{CHRG_FAULT}
- D2 pad 1: SOLAR_PRE_INH -> /Connectors/VSOLAR_IN
- D3 pad 1: SOLAR_PRE_INH -> /Connectors/VSOLAR_IN
- D5 pad 2: EDFA_5V_S -> 5V_2_S
- D7 pad 2: 5V_S -> 5V_1_S
- D8 pad 2: /EDFA_5V -> EDFA_5V
- J1 pad 1: unconnected-(J1-Pin_1-Pad1) -> LDO_3V3
- J1 pad 2: unconnected-(J1-Pin_2-Pad2) -> /Control/SWDIO
- J1 pad 3: unconnected-(J1-Pin_3-Pad3) -> /Control/SWCLK
- J1 pad 4: unconnected-(J1-Pin_4-Pad4) -> /Control/~{RESET}
- J1 pad 5: unconnected-(J1-Pin_5-Pad5) -> GND
- J2 pad 1: unconnected-(J2-Pin_1-Pad1) -> /Connectors/CAN_L
- J2 pad 21: unconnected-(J2-Pin_21-Pad21) -> EDFA_5V
- J2 pad 22: /~{CHRG_FAULT} -> EDFA_5V
- J2 pad 24: /~{CHRG_STAT} -> unconnected-(J2-Pin_24-Pad24)
- J2 pad 28: ENAB_BURN_1 -> unconnected-(J2-Pin_28-Pad28)
- J2 pad 29: BURN_FET -> unconnected-(J2-Pin_29-Pad29)
- J2 pad 3: unconnected-(J2-Pin_3-Pad3) -> /Connectors/CAN_H
- J2 pad 30: ENAB_BURN_2 -> unconnected-(J2-Pin_30-Pad30)
- J2 pad 31: /5V_S_EN -> unconnected-(J2-Pin_31-Pad31)
- J2 pad 34: 3V3_S -> unconnected-(J2-Pin_34-Pad34)
- J2 pad 36: /ADJ -> unconnected-(J2-Pin_36-Pad36)
- J2 pad 37: /KAPTON_EN -> 3V3_S
- J2 pad 38: /BATT_THERM_R -> 3V3_S
- J2 pad 39: /3V3_S_EN -> 5V_2_S
- J2 pad 40: /EDFA_5V_EN -> 5V_2_S
- J2 pad 41: SDA -> unconnected-(J2-Pin_41-Pad41)
- J2 pad 42: /EDFA_5V_S -> unconnected-(J2-Pin_42-Pad42)
- J2 pad 43: SCL -> unconnected-(J2-Pin_43-Pad43)
- J2 pad 44: /EDFA_5V_S -> unconnected-(J2-Pin_44-Pad44)
- J2 pad 45: /5V_S -> 5V_1_S
- J2 pad 46: /5V_S -> 5V_1_S
- J2 pad 5: /VBATT_IN -> unconnected-(J2-Pin_5-Pad5)
- J2 pad 6: /VBATT_IN -> unconnected-(J2-Pin_6-Pad6)
- J2 pad 7: /VBATT_IN -> unconnected-(J2-Pin_7-Pad7)
- J2 pad 8: /VBATT_IN -> unconnected-(J2-Pin_8-Pad8)
- J3 pad 1: SOLAR_PRE_INH -> /Connectors/BATT_CS
- J3 pad 2: VINA -> Net-(J3-Pin_2)
- J4 pad 1: /VBATT_PRE_INH -> Net-(J3-Pin_2)
- J4 pad 2: /BATT_CS -> /Connectors/VBATT_PRE_INH
- J7 pad 19: EDFA_5V_STAT -> unconnected-(J7-Pin_19-Pad19)
- J7 pad 2: /PDU_TEMP -> /Connectors/PDU_TEMP
- J7 pad 23: 5V_STAT -> unconnected-(J7-Pin_23-Pad23)
- J7 pad 24: 3V3_STAT -> unconnected-(J7-Pin_24-Pad24)
- J7 pad 33: 3V3_S -> unconnected-(J7-Pin_33-Pad33)
- J7 pad 47: unconnected-(J7-Pin_47-Pad47) -> VBATT
- L1 pad 1: GND -> GND_REF
- L2 pad 2: /EDFA_5V -> EDFA_5V
- Q2 pad 1: /VBATT_IN -> /Connectors/VBATT_IN
- Q2 pad 3: /VBATT_PRE_INH -> /Connectors/VBATT_PRE_INH
- Q3 pad 2: BURN_FET -> /Control/MASTER_BURN_EN
- R2 pad 2: /VBATT_IN -> /Connectors/VBATT_IN
- R21 pad 1: /EDFA_5V -> Net-(U11-~{RESET})
- R21 pad 2: EDFA_5V_STAT -> /Control/~{RESET}
- R22 pad 2: /EDFA_5V -> EDFA_5V
- R25 pad 1: GND -> Net-(D4-K)
- R25 pad 2: Net-(D4-K) -> GND
- R26 pad 1: GND -> VBATT
- R26 pad 2: Net-(D5-K) -> Net-(U14-ADJ)
- R28 pad 1: GND -> Net-(U14-ADJ)
- R28 pad 2: Net-(D7-K) -> GND
- R3 pad 1: /BATT_CS -> /Sensors/BATT_CS
- R30 pad 1: GND -> LDO_3V3
- R30 pad 2: Net-(D9-K) -> /Control/SWCLK
- R32 pad 1: BURN_FET -> /Control/MASTER_BURN_EN
- R34 pad 1: ENAB_BURN_1 -> /Control/BURN_1_PWM
- R35 pad 1: ENAB_BURN_2 -> /Control/BURN_2_PWM
- R37 pad 2: ENAB_BURN_1 -> /Control/BURN_1_PWM
- R38 pad 2: ENAB_BURN_2 -> /Control/BURN_2_PWM
- R42 pad 1: /ADJ -> Net-(D7-K)
- R42 pad 2: VBATT -> GND
- R43 pad 1: GND -> Net-(D5-K)
- R43 pad 2: /ADJ -> GND
- R5 pad 1: /BATT_CS -> /Sensors/BATT_CS
- TP1 pad 1: /EDFA_5V -> EDFA_5V
- U1 pad 1: /PDU_TEMP -> (no net)
- U1 pad 2: unconnected-(U1-NC_2-Pad2) -> (no net)
- U1 pad 3: unconnected-(U1-NC_3-Pad3) -> (no net)
- U1 pad 4: GND -> (no net)
- U1 pad 5: 3V3 -> (no net)
- U1 pad 6: unconnected-(U1-NC_4-Pad6) -> (no net)
- U1 pad 7: unconnected-(U1-NC-Pad7) -> (no net)
- U1 pad 8: 3V3 -> (no net)
- U10 pad 1: EDFA_5V_S -> 5V_2_S
- U10 pad 2: EDFA_5V -> 5V
- U10 pad 3: EDFA_5V -> 5V
- U10 pad 4: EDFA_5V_EN -> /Control/5V_2_S_EN
- U10 pad 5: GND -> Net-(D5-K)
- U10 pad 6: EDFA_5V -> 5V
- U10 pad 7: EDFA_5V -> 5V
- U10 pad 8: EDFA_5V_S -> 5V_2_S
- U12 pad 1: 5V_S -> 5V_1_S
- U12 pad 4: 5V_S_EN -> /Control/5V_1_S_EN
- U12 pad 5: GND -> Net-(D7-K)
- U12 pad 8: 5V_S -> 5V_1_S
- U14 pad H7: /ADJ -> Net-(U14-ADJ)
- U14 pad J7: /~{CHRG_FAULT} -> /Charging/~{CHRG_FAULT}
- U14 pad K7: /~{CHRG_STAT} -> /Charging/~{CHRG_STAT}
- U15 pad 1: MRAM_CS -> /Control/MRAM_CS
- U15 pad 2: MISO -> /Control/MISO
- U15 pad 3: WRITE_PROT -> /Control/WP
- U15 pad 5: MOSI -> /Control/MOSI
- U15 pad 6: SCK -> /Control/SCK
- U15 pad 7: HOLD -> /Control/HOLD
- U15 pad 8: 3V3 -> LDO_3V3
- U19 pad 1: unconnected-(U19-VBAT-Pad1) -> LDO_3V3
- U19 pad 11: unconnected-(U19-PA1-Pad11) -> /Control/SCK
- U19 pad 14: unconnected-(U19-PA4-Pad14) -> /Control/HOLD
- U19 pad 15: unconnected-(U19-PA5-Pad15) -> /Control/WP
- U19 pad 16: unconnected-(U19-PA6-Pad16) -> /Control/MISO
- U19 pad 17: unconnected-(U19-PA7-Pad17) -> /Control/MOSI
- U19 pad 18: unconnected-(U19-PB0-Pad18) -> /Charging/~{CHRG_STAT}
- U19 pad 19: unconnected-(U19-PB1-Pad19) -> /Charging/~{CHRG_FAULT}
- U19 pad 20: unconnected-(U19-PB2-Pad20) -> /Control/EDFA_5V_EN
- U19 pad 21: unconnected-(U19-PB10-Pad21) -> /Control/BURN_1_PWM
- U19 pad 22: unconnected-(U19-PB11-Pad22) -> /Control/EDFA_5V_PG
- U19 pad 23: Net-(U19-VSS-Pad23) -> GND
- U19 pad 24: unconnected-(U19-VDD-Pad24) -> LDO_3V3
- U19 pad 25: unconnected-(U19-PB12-Pad25) -> /Control/5V_PG
- U19 pad 26: unconnected-(U19-PB13-Pad26) -> /Control/3V3_PG
- U19 pad 28: unconnected-(U19-PB15-Pad28) -> /Control/WDI
- U19 pad 29: unconnected-(U19-PA8-Pad29) -> /Control/MRAM_CS
- U19 pad 30: unconnected-(U19-PA9-Pad30) -> /Control/SCL
- U19 pad 31: unconnected-(U19-PA10-Pad31) -> /Control/SDA
- U19 pad 32: unconnected-(U19-PA11-Pad32) -> /Control/CAN_TX
- U19 pad 33: unconnected-(U19-PA12-Pad33) -> /Control/CAN_RX
- U19 pad 34: unconnected-(U19-PA13-Pad34) -> /Control/SWDIO
- U19 pad 35: Net-(U19-VSS-Pad23) -> GND
- U19 pad 36: unconnected-(U19-VDD-Pad36) -> LDO_3V3
- U19 pad 37: unconnected-(U19-PA14-Pad37) -> /Control/SWCLK
- U19 pad 39: unconnected-(U19-PB3-Pad39) -> /Control/5V_EN
- U19 pad 40: unconnected-(U19-PB4-Pad40) -> /Control/3V3_EN
- U19 pad 41: unconnected-(U19-PB5-Pad41) -> /Control/5V_2_S_EN
- U19 pad 42: unconnected-(U19-PB6-Pad42) -> /Control/5V_1_S_EN
- U19 pad 43: unconnected-(U19-PB7-Pad43) -> /Control/3V3_S_EN
- U19 pad 45: unconnected-(U19-PB8-Pad45) -> /Control/BURN_2_PWM
- U19 pad 46: unconnected-(U19-PB9-Pad46) -> /Control/MASTER_BURN_EN
- U19 pad 47: Net-(U19-VSS-Pad23) -> GND
- U19 pad 48: unconnected-(U19-VDD-Pad48) -> LDO_3V3
- U19 pad 5: unconnected-(U19-PH0-Pad5) -> /Control/HSE_IN
- U19 pad 6: unconnected-(U19-PH1-Pad6) -> /Control/HSE_OUT
- U19 pad 7: unconnected-(U19-NRST-Pad7) -> /Control/~{RESET}
- U19 pad 8: unconnected-(U19-VSSA-Pad8) -> GND
- U19 pad 9: unconnected-(U19-VDDA-Pad9) -> Net-(U19-VDDA)
- U2 pad 2: SDA -> /Control/SDA
- U2 pad 3: SDA -> /Control/SDA
- U2 pad 4: SCL -> /Control/SCL
- U2 pad 5: 3V3_S -> 3V3
- U3 pad 3: SDA -> /Control/SDA
- U3 pad 4: SCL -> /Control/SCL
- U3 pad 5: 3V3_S -> 3V3
- U4 pad 2: SCL -> /Control/SCL
- U4 pad 3: SDA -> /Control/SDA
- U4 pad 4: SCL -> /Control/SCL
- U4 pad 5: 3V3_S -> 3V3
- U5 pad 1: SDA -> /Control/SDA
- U5 pad 3: SDA -> /Control/SDA
- U5 pad 4: SCL -> /Control/SCL
- U5 pad 5: 3V3_S -> 3V3
- U6 pad 14: /EDFA_5V -> EDFA_5V
- U6 pad 15: EDFA_5V_STAT -> /Control/EDFA_5V_PG
- U6 pad 4: VBATT -> /Control/EDFA_5V_EN
- U7 pad 15: 3V3_STAT -> /Control/3V3_PG
- U7 pad 4: VBATT -> /Control/3V3_EN
- U8 pad 15: 5V_STAT -> /Control/5V_PG
- U8 pad 4: VBATT -> /Control/5V_EN
- U9 pad 4: 3V3_S_EN -> /Control/3V3_S_EN
- U9 pad 5: GND -> Net-(D4-K)
Routing:
- net (no net): track 87.3 -> 777.6 mm, vias 6 -> 26
- net /~{CHRG_FAULT}: track 95.4 -> 0.00 mm, vias 3 -> 0
- net /~{CHRG_STAT}: track 93.5 -> 0.00 mm, vias 3 -> 0
- net unconnected-(J2-Pin_41-Pad41): track 0.00 -> 82.8 mm, vias 0 -> 2
- net SDA: track 82.8 -> 0.00 mm, vias 2 -> 0
- net 5V_STAT: track 80.2 -> 0.00 mm, vias 2 -> 0
- net /KAPTON_EN: track 79.0 -> 0.00 mm
- net unconnected-(J2-Pin_43-Pad43): track 0.00 -> 77.1 mm, vias 0 -> 3
- net SCL: track 77.1 -> 0.00 mm, vias 3 -> 0
- net EDFA_5V_STAT: track 71.2 -> 0.00 mm, vias 2 -> 0
- net 5V_S_EN: track 66.5 -> 0.00 mm, vias 1 -> 0
- net /Control/5V_1_S_EN: track 0.00 -> 66.5 mm, vias 0 -> 1
- net ENAB_BURN_1: track 66.5 -> 0.00 mm, vias 2 -> 0
- net 3V3: track 71.4 -> 134.7 mm, vias 9 -> 13
- net 3V3_STAT: track 62.2 -> 0.00 mm, vias 1 -> 0
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- added copper zone on F.Cu, net /Connectors/VBATT_PRE_INH
- added copper zone on In2.Cu, net 5V_1_S
- added copper zone on In2.Cu, net 5V_2_S
- removed copper zone on F.Cu, net /BATT_CS
- removed copper zone on F.Cu, net /VBATT_IN
- removed copper zone on In2.Cu, net 5V_S
- removed copper zone on In2.Cu, net EDFA_5V_S
- removed copper zone on B.Cu, net GND_REF
- removed copper zone on F.Cu, net GND_REF
