File: flight-subsystem-designs/power/power-distribution/PowerDistribution.kicad_pcb (KiCad board)
At the start: 4 copper layers, 90.2 x 96 mm, 202 parts, among them J1 Conn_01x05, J10 Molex 205338-4, J11 Conn_01x02, J12 Conn_01x02, J14 Molex 205338-2, J15 Battery Header, J2 Conn_02x26_Odd_Even, J3 Molex 205338-2, J4 Molex 205338-2, J5 Molex 205338-2, J6 Molex 205338-2, J7 Conn_02x26_Odd_Even, J8 Molex 205338-4, J9 Molex 205338-4, Q1 NMOS, Q2 NMOS, Q3 BC848ALT1G, Q4 IRLML2803PBFCT, Q5 IRLML2803PBFCT, Q6 NMOS, Q7 NMOS, SW1 SW_Push, U1 TMP36FSZ, U10 LTC1477CS8, U11 MAX706RESA, U12 LTC1477CS8, U13 SI4835DDY, U14 LTM8062AIV-PBF, U15 MR25H256ACDF, U16 TCAN337G, U17 SI3407DV, U18 SI3407DV, U19 STM32L431CBT6, U2 INA219AIDR, U20 LT1761-3.3, U3 INA219AIDR, U4 INA219AIDR, U5 INA219AIDR, U6 LT8610, U7 LT8610, U8 LT8610, U9 LTC1477CS8, Y1 16 MHz

Commit message: shi
Parts:
- removed C38: 4.7uF, Capacitor_SMD:C_1206_3216Metric
- removed C48: 10pF, Capacitor_SMD:C_0603_1608Metric
- removed C54: 22uF, Capacitor_SMD:C_0805_2012Metric
- removed C55: 0.1uF, Capacitor_SMD:C_0805_2012Metric
- removed C56: 4.7uF, Capacitor_Tantalum_SMD:CP_EIA-3528-12_Kemet-T
- removed D19: RED, LED_SMD:LED_0603_1608Metric
- removed J14, J3, J4, J5, J6: Molex 205338-2, Connector_Molex:Molex_Pico-Lock_205338-0002_1x02-1MP_P2.00mm_Horizontal
- removed JP1, JP2, JP3, JP4, JP5: Jumper_2_Open, Jumper:SolderJumper-2_P1.3mm_Open_TrianglePad1.0x1.5mm
- removed L1, L5: AIMC-0805-2N2S-T, Inductor_SMD:L_0805_2012Metric
- removed Q1, Q2, Q6, Q7: NMOS, Package_TO_SOT_SMD:TSOT-23
- removed R55: 1M, Resistor_SMD:R_0603_1608Metric
- removed R60, R61, R62: 10k, Resistor_SMD:R_0603_1608Metric
- removed R63: 150, Resistor_SMD:R_0603_1608Metric
- removed Y1: 16 MHz, Crystal:Crystal_SMD_3225-4Pin_3.2x2.5mm
- added C39: 0.1uF, Capacitor_SMD:C_0603_1608Metric, F.Cu at (206.8, 96.0)
- added J13: RBF, Connector_Molex:Molex_PicoBlade_53047-0210_1x02_P1.25mm_Vertical, F.Cu at (251.8, 97.8)
- added J16: NO, Connector_Molex:Molex_PicoBlade_53047-0210_1x02_P1.25mm_Vertical, F.Cu at (251.8, 91.6)
- added J17: NO, Connector_Molex:Molex_PicoBlade_53047-0210_1x02_P1.25mm_Vertical, F.Cu at (251.8, 86.2)
- added J18: NC, Connector_Molex:Molex_PicoBlade_53047-0210_1x02_P1.25mm_Vertical, F.Cu at (251.7, 128.3)
- added J19: RBF, Connector_Molex:Molex_PicoBlade_53047-0210_1x02_P1.25mm_Vertical, F.Cu at (173.0, 103.5)
- added Q8: PMOS, Package_SO:TSOP-6_1.65x3.05mm_P0.95mm, F.Cu at (248.0, 97.6)
- added Q9: NMOS, Package_SO:TSOP-6_1.65x3.05mm_P0.95mm, F.Cu at (247.9, 128.2)
- added R44: 50, Resistor_SMD:R_0603_1608Metric, F.Cu at (207.2, 91.0)
- added R64: 100k, Resistor_SMD:R_0603_1608Metric, F.Cu at (247.7, 100.3)
- added R65: 100k, Resistor_SMD:R_0603_1608Metric, F.Cu at (247.9, 130.8)
- added R66: 100k, Resistor_SMD:R_0603_1608Metric, F.Cu at (176.4, 101.0)
- added U21: SIT2024B, Package_TO_SOT_SMD:SOT-23-5, F.Cu at (205.1, 94.2)
- added U22: SI3407DV, Package_SO:TSOP-6_1.65x3.05mm_P0.95mm, F.Cu at (176.7, 103.7)
- C10, C11, C8: value 0.1UF -> 0.1uF
- C2: value 0.1uF -> 4.7uF; footprint Capacitor_SMD:C_0805_2012Metric -> Capacitor_SMD:C_1206_3216Metric
- C3: value 22uF -> 4.7uF; footprint Capacitor_SMD:C_0805_2012Metric -> Capacitor_Tantalum_SMD:CP_EIA-3528-12_Kemet-T
- C33, C6, D2, R10, R13, R29, R31, R45, R46, R7, U4: moved to F.Cu
- C47: value 10pF -> 0.1uF
- C9: value 0.1UF -> 0.1uF; moved to F.Cu
- D18: value RED -> GREEN
- J1: footprint Connector_PinHeader_2.54mm:PinHeader_1x05_P2.54mm_Vertical -> Connector_Molex:Molex_PicoBlade_53047-0510_1x05_P1.25mm_Vertical
- J10, J8: footprint Connector_Molex:Molex_Pico-Lock_205338-0004_1x04-1MP_P2.00mm_Horizontal -> Connector_Molex:Molex_PicoBlade_53047-0410_1x04_P1.25mm_Vertical
- J11, J12: footprint Connector_Molex:Molex_Pico-Lock_205338-0002_1x02-1MP_P2.00mm_Horizontal -> Connector_Molex:Molex_PicoBlade_53047-0210_1x02_P1.25mm_Vertical
- J9: footprint Connector_Molex:Molex_Pico-Lock_205338-0004_1x04-1MP_P2.00mm_Horizontal -> Connector_Molex:Molex_PicoBlade_53047-0410_1x04_P1.25mm_Vertical; moved to F.Cu
- R1, R2, R54: value 1M -> 150
- R25: value 150 -> 10k; moved to F.Cu
- R42, R43: value 150 -> 10k
- moved TP7 146.4 mm to (172.4, 98.4)
- moved C46 146.2 mm to (231.2, 100.0), turned to 90 degrees
- moved R49 133.7 mm to (174.2, 87.9)
- moved U15 132.8 mm to (226.7, 101.3)
- moved R48 130.1 mm to (174.2, 65.5)
- moved R56 129.9 mm to (174.2, 76.7)
- moved D13 129.7 mm to (235.9, 81.8)
- moved J1 129.4 mm to (215.5, 66.8), turned to 180 degrees
- moved D14 127.1 mm to (242.9, 141.7)
- moved R57 126.7 mm to (176.1, 121.9)
- moved U11 126.5 mm to (199.2, 101.4), turned to 180 degrees
- moved R27 116.9 mm to (175.9, 129.7), turned to 180 degrees
- moved D18 116.6 mm to (212.8, 79.8), turned to -135 degrees
- moved R21 116.1 mm to (198.4, 91.8), turned to 90 degrees
- moved SW1 116.0 mm to (197.5, 85.5)
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Connections:
- C1 pad 2: 3V3 -> LDO_3V3
- C2 pad 1: GND_REF -> GND
- C2 pad 2: /Connectors/VBATT_IN -> Net-(C2-Pad2)
- C28 pad 2: Net-(D4-K) -> GND
- C29 pad 1: 5V_2_S -> 5V_1_S
- C29 pad 2: Net-(D5-K) -> GND
- C3 pad 1: GND_REF -> VBATT
- C3 pad 2: /Connectors/VBATT_IN -> GND
- C31 pad 1: 5V_1_S -> 5V_2_S
- C31 pad 2: Net-(D7-K) -> GND
- C47 pad 1: /Control/HSE_IN -> GND
- C47 pad 2: GND -> LDO_3V3
- D15 pad 2: /Connectors/VSOLAR_IN -> /Connectors/sol_1_diode
- D16 pad 2: /Connectors/VSOLAR_IN -> /Connectors/sol_2_diode
- D17 pad 2: /Connectors/VSOLAR_IN -> /Connectors/sol_3_diode
- D18 pad 2: /Connectors/VSOLAR_MPPT -> Net-(D18-A)
- D5 pad 2: 5V_2_S -> 5V_1_S
- D7 pad 2: 5V_1_S -> 5V_2_S
- R1 pad 1: Net-(Q1-S) -> GND
- R1 pad 2: Net-(J6-Pin_1) -> Net-(D11-K)
- R2 pad 1: Net-(Q1-D) -> GND
- R2 pad 2: /Connectors/VBATT_IN -> Net-(D12-K)
- R25 pad 1: Net-(D4-K) -> /Control/3V3_S_EN
- R3 pad 1: /Sensors/BATT_CS -> /Connectors/BATT_CS
- R42 pad 1: Net-(D7-K) -> /Control/5V_1_S_EN
- R43 pad 1: Net-(D5-K) -> /Control/5V_2_S_EN
- R45 pad 1: GND -> Net-(D4-K)
- R45 pad 2: Net-(D11-K) -> GND
- R46 pad 1: GND -> Net-(D5-K)
- R46 pad 2: Net-(D12-K) -> GND
- R5 pad 1: /Sensors/BATT_CS -> /Connectors/BATT_CS
- R50 pad 1: GND -> Net-(D7-K)
- R50 pad 2: Net-(D18-K) -> GND
- R54 pad 1: Net-(Q6-S) -> Net-(D18-K)
- R54 pad 2: Net-(J14-Pin_1) -> GND
- U1 pad 1: (no net) -> /Connectors/PDU_TEMP
- U1 pad 2: (no net) -> unconnected-(U1-NC_2-Pad2)
- U1 pad 3: (no net) -> unconnected-(U1-NC_3-Pad3)
- U1 pad 4: (no net) -> GND
- U1 pad 5: (no net) -> LDO_3V3
- U1 pad 6: (no net) -> unconnected-(U1-NC_4-Pad6)
- U1 pad 7: (no net) -> unconnected-(U1-NC-Pad7)
- U1 pad 8: (no net) -> LDO_3V3
- U10 pad 1: 5V_2_S -> 5V_1_S
- U10 pad 4: /Control/5V_2_S_EN -> /Control/5V_1_S_EN
- U10 pad 5: Net-(D5-K) -> GND
- U10 pad 8: 5V_2_S -> 5V_1_S
- U12 pad 1: 5V_1_S -> 5V_2_S
- U12 pad 4: /Control/5V_1_S_EN -> /Control/5V_2_S_EN
- U12 pad 5: Net-(D7-K) -> GND
- U12 pad 8: 5V_1_S -> 5V_2_S
- U14 pad K1: Net-(C38-Pad2) -> Net-(C2-Pad2)
- U14 pad K2: Net-(C38-Pad2) -> Net-(C2-Pad2)
- U14 pad K3: Net-(C38-Pad2) -> Net-(C2-Pad2)
- U14 pad L1: Net-(C38-Pad2) -> Net-(C2-Pad2)
- U14 pad L2: Net-(C38-Pad2) -> Net-(C2-Pad2)
- U14 pad L3: Net-(C38-Pad2) -> Net-(C2-Pad2)
- U19 pad 12: unconnected-(U19-PA2-Pad12) -> /Control/EDFA_5V_PG
- U19 pad 13: unconnected-(U19-PA3-Pad13) -> /Control/5V_PG
- U19 pad 18: /Charging/~{CHRG_STAT} -> /Charging/~{CHRG_FAULT}
- U19 pad 19: /Charging/~{CHRG_FAULT} -> /Charging/~{CHRG_STAT}
- U19 pad 20: /Control/EDFA_5V_EN -> /Control/MRAM_CS
- U19 pad 21: /Control/BURN_1_PWM -> /Control/5V_1_S_EN
- U19 pad 22: /Control/EDFA_5V_PG -> /Control/EDFA_5V_EN
- U19 pad 25: /Control/5V_PG -> /Control/5V_2_S_EN
- U19 pad 26: /Control/3V3_PG -> /Control/5V_EN
- U19 pad 27: unconnected-(U19-PB14-Pad27) -> /Control/BURN_2_PWM
- U19 pad 28: /Control/WDI -> /Control/MASTER_BURN_EN
- U19 pad 29: /Control/MRAM_CS -> /Control/BURN_1_PWM
- U19 pad 38: unconnected-(U19-PA15-Pad38) -> Net-(D18-A)
- U19 pad 39: /Control/5V_EN -> unconnected-(U19-PB3-Pad39)
- U19 pad 40: /Control/3V3_EN -> /Control/3V3_PG
- U19 pad 41: /Control/5V_2_S_EN -> /Control/3V3_EN
- U19 pad 42: /Control/5V_1_S_EN -> /Control/3V3_S_EN
- U19 pad 43: /Control/3V3_S_EN -> /Control/WDI
- U19 pad 45: /Control/BURN_2_PWM -> unconnected-(U19-PB8-Pad45)
- U19 pad 46: /Control/MASTER_BURN_EN -> unconnected-(U19-PB9-Pad46)
- U19 pad 6: /Control/HSE_OUT -> unconnected-(U19-PH1-Pad6)
- U9 pad 5: Net-(D4-K) -> GND
Routing:
- net (no net): track 777.6 -> 0.00 mm, vias 26 -> 0
- net 3V3_S: track 154.6 -> 13.0 mm, vias 3 -> 2
- net /Control/SCL: track 0.00 -> 109.6 mm, vias 0 -> 6
- net /Control/SDA: track 0.00 -> 106.6 mm, vias 0 -> 6
- net 3V3: track 134.7 -> 41.9 mm, vias 13 -> 11
- net unconnected-(J2-Pin_41-Pad41): track 82.8 -> 0.00 mm, vias 2 -> 0
- net unconnected-(J2-Pin_43-Pad43): track 77.1 -> 0.00 mm, vias 3 -> 0
- net /Control/3V3_EN: track 0.00 -> 69.6 mm, vias 0 -> 2
- net LDO_3V3: track 0.00 -> 66.5 mm, vias 0 -> 13
- net /Control/3V3_PG: track 0.00 -> 60.5 mm, vias 0 -> 2
- net /Control/EDFA_5V_EN: track 0.00 -> 57.5 mm, vias 0 -> 2
- net GND: track 104.4 -> 160.1 mm, vias 75 -> 86
- net /Control/~{RESET}: track 0.00 -> 48.8 mm, vias 0 -> 2
- net /Control/3V3_S_EN: track 0.00 -> 47.5 mm, vias 0 -> 2
- net /Control/5V_EN: track 0.00 -> 44.3 mm, vias 0 -> 2
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- added copper zone on F.Cu, net /Connectors/BATT_CS
- added copper zone on F.Cu, net /Connectors/SOLAR_IN_+Y
- added copper zone on F.Cu, net /Connectors/VBATT_IN
- added copper zone on F.Cu, net /Connectors/VSOLAR_IN
- added copper zone on In2.Cu, net /Connectors/VSOLAR_IN
- added copper zone on F.Cu, net /Connectors/sol_2_diode
- added copper zone on F.Cu, net GND_REF
- added copper zone on F.Cu, net LDO_3V3
- added copper zone on In2.Cu, net LDO_3V3
- added copper zone on F.Cu, net Net-(C2-Pad2)
- removed copper zone on In2.Cu, net (none)
- removed copper zone on B.Cu, net /Connectors/SOLAR_IN_+Y
- removed copper zone on F.Cu, net /Connectors/VBATT_PRE_INH
- removed copper zone on B.Cu, net /Connectors/sol_2_diode
- removed copper zone on F.Cu, net /Deployment/b1
- removed copper zone on F.Cu, net /Deployment/b2
- removed copper zone on F.Cu, net Net-(C38-Pad2)
- removed copper zone on B.Cu, net VINA
Other:
- outline, holes or cut-outs redrawn
- board text added: "power control & distribution unit"
- board text added: "rev. 4.0, 05.12.26"
- board text removed: "(this one's for you, Ian)"
- board text removed: "3V3 Bus"
- board text removed: "3V3 Switch"
- board text removed: "5V Bus"
- board text removed: "5V Switch"
- board text removed: "Batt Heat"
- board text removed: "Burn Wire"
- board text removed: "Chg Fault"
- board text removed: "EDFA Bus"
- board text removed: "EDFA Switch"
- board text removed: "Heat"
- board text removed: "Inhibit Switches"
- board text removed: "Solar Chg"
- board text removed: "power distribution unit"
- board text removed: "rev. 3.0.0, 06.30.25"
- board text removed: "{dblquote}I really get motivated when I have doubters{dblquote} - Shaquille O'Neal"
